File: Remote Switch v3/ReceiverController/receiver.brd (EAGLE design)
At the start: 42 x 42 mm, 40 parts, among them IC1 LNK304, IC2 MCP1703CB, IC3 STM8L101F2, J1 POWER_CONN_4, T1 BT136

Commit message: PCB work
Parts:
- moved C5 9.34 mm to (55.1, 24.4)
- moved LED1 7.97 mm to (46.7, 3.30)
- moved C10 7.97 mm to (33.5, 4.14)
- moved C6 7.97 mm to (30.7, 14.5)
- moved C9 7.97 mm to (35.5, 4.12)
- moved R3 7.97 mm to (36.6, 16.6)
- moved T1 7.97 mm to (35.3, 26.7)
- moved B1 7.97 mm to (23.5, 35.1)
- moved C2 7.97 mm to (14.1, 6.36)
- moved C4 7.97 mm to (20.4, 26.8)
- moved R13 7.97 mm to (18.8, 9.18)
- moved R5 7.97 mm to (12.8, 24.6)
- moved S1 7.97 mm to (14.5, 11.8)
- moved C12 7.97 mm to (14.5, 16.7)
- moved R7 7.97 mm to (11.7, 19.7)
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Routing:
- net GND: track 89.1 -> 112.5 mm
- net RF_DATA: track 10.4 -> 18.3 mm
- net +3V3: track 34.8 -> 42.1 mm
Other:
- board size 42 x 42 mm -> 50 x 42 mm

Commit message: PCB work
Parts:
- added C13: 100n, resistor:C0603K
- moved D1 42.3 mm to (13.8, 19.5), turned to 180 degrees
- moved C5 34.8 mm to (20.8, 18.5)
- moved R10 33.8 mm to (4.64, 23.6), turned to 90 degrees
- moved C8 26.0 mm to (9.42, 14.1), turned to 270 degrees
- moved IC2 25.1 mm to (15.0, 15.7)
- moved C6 25.1 mm to (5.89, 18.5), turned to 0 degrees
- moved D2 24.0 mm to (4.65, 28.3), turned to 90 degrees
- moved C11 22.8 mm to (18.1, 13.7), turned to 270 degrees
- moved OK1 15.9 mm to (28.4, 15.9), flipped to the bottom, turned to 0 degrees
- moved L1 14.6 mm to (10.3, 26.2), turned to 270 degrees
- moved R6 13.7 mm to (34.2, 19.0), turned to 0 degrees
- moved C10 12.5 mm to (45.8, 6.56), turned to 270 degrees
- moved C7 12.0 mm to (38.0, 1.99)
- moved IC3 12.0 mm to (38.5, 7.24)
- moved R2 12.0 mm to (41.6, 2.04)
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Connections:
- removed net N$19: B1.AC1, R1.1
- new net N$10: B1.AC2, R1.1
- net +5V: now also C13.1
- net GND: now also C13.2
- net N: now also B1.AC1; no longer B1.AC2
Routing:
- net GND: track 112.5 -> 153.6 mm, vias 4 -> 5
- net +3V3: track 42.1 -> 74.6 mm, vias 8 -> 6
- net N$8: track 32.3 -> 9.38 mm
- net +5V: track 5.06 -> 25.3 mm
- net N$3: track 0.00 -> 15.1 mm
- net SWIM: track 17.1 -> 29.7 mm
- net RST: track 15.3 -> 27.3 mm
- net N$9: track 4.74 -> 16.7 mm
- net LED_TX_ERR2: track 20.0 -> 9.71 mm
- net LOAD: track 40.1 -> 30.5 mm
- net N$19: track 9.19 -> 0.00 mm
- net N$1: track 5.24 -> 12.8 mm
- net N$10: track 0.00 -> 7.53 mm
- net N$11: track 2.95 -> 9.34 mm
- net N$2: track 16.9 -> 11.5 mm
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Other:
- board text added: "MOC3063"

Commit message: PCB work
Parts:
- IC1: device comp_RFSwitch_v3:SO8 -> comp_RFSwitch_v3:SO8_NO_PIN3
Routing:
- net LOAD: track 30.5 -> 25.7 mm
Changed lines of the file:
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@@
 <element name="R1" library="resistor" package="0309/10" value="10" x="21.69" y="39.446" rot="MR180"/>
 <element name="C10" library="resistor" package="C0805K" value="2.2u" x="45.83" y="6.561" rot="R270"/>
-<element name="IC1" library="comp_RFSwitch_v3" package="SO8" value="LNK304" x="17.89" y="28.166" rot="R90"/>
+<element name="IC1" library="comp_RFSwitch_v3" package="SO8_NO_PIN3" value="LNK304" x="17.89" y="28.166" rot="R90"/>
 <element name="D2" library="comp_RFSwitch_v3" package="DO214-AC" value="US1G-DIO" x="4.648" y="28.253" rot="R90"/>
 <element name="L1" library="comp_RFSwitch_v3" package="DE0703" value="FERROCORE_DE0703-1000" x="10.307" y="26.241" rot="R270"/>
@@
 <vertex x="44.336" y="31.377"/>
 </polygon>
-<wire x1="35.174" y1="18.998" x2="35.174" y2="26.628" width="1.016" layer="1"/>
 <wire x1="35.174" y1="26.628" x2="35.198" y2="26.652" width="1.016" layer="1" curve="-90"/>
+<wire x1="35.174" y1="18.998" x2="37.875" y2="18.998" width="1.016" layer="1"/>
+<wire x1="37.875" y1="18.998" x2="37.875" y2="18.927" width="1.016" layer="1"/>
 </signal>
 <signal name="N$9">

Commit message: PCB work
Parts:
- removed SIG_1, SIG_2, SIG_3, SIG_4: CON_PAD, componente_RFSwitch:SMD_PAD
- added JP1: (no value), pinhead:1X04
- moved RF1 40.8 mm to (30.9, 2.10), flipped to the bottom, turned to 0 degrees
- moved R9 3.56 mm to (20.9, 5.86), turned to 270 degrees
- moved R13 1.41 mm to (7.55, 8.83)
- moved OK1 1.41 mm to (27.4, 16.9)
- moved B1 1.41 mm to (18.8, 36.0)
- moved C1 1.41 mm to (4.76, 9.04)
- moved C10 1.41 mm to (44.8, 7.56)
- moved C11 1.41 mm to (17.1, 14.7)
- moved C12 1.41 mm to (17.3, 9.30)
- moved C13 1.41 mm to (10.9, 16.5)
- moved C2 1.41 mm to (2.75, 9.05)
- moved C3 1.41 mm to (8.81, 36.9)
- moved C4 1.41 mm to (16.0, 25.5)
- moved C5 1.41 mm to (19.8, 19.5)
- moved C6 1.41 mm to (4.89, 19.5)
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Connections:
- net +3V3: now also JP1.1; no longer SIG_1.P$1
- net GND: now also JP1.3; no longer SIG_3.P$1
- net RST: now also JP1.4; no longer SIG_4.P$1
- net SWIM: now also JP1.2; no longer SIG_2.P$1
Routing:
- net GND: track 153.6 -> 110.2 mm, vias 5 -> 4
- net +3V3: track 74.6 -> 48.3 mm, vias 6 -> 4
- net RF_DATA: track 18.3 -> 0.00 mm
- net RST: track 27.3 -> 15.8 mm
- net SWIM: track 29.7 -> 19.2 mm, vias 2 -> 1
Other:
- outline, holes or cut-outs redrawn

Commit message: PCB work
Parts:
- moved C2 12.0 mm to (13.3, 3.37), flipped to the bottom, turned to 270 degrees
- moved C1 12.0 mm to (15.4, 3.61), flipped to the bottom, turned to 270 degrees
- moved D2 7.75 mm to (4.41, 21.5), turned to 180 degrees
- moved C6 3.83 mm to (5.31, 15.7), turned to 90 degrees
- moved R10 2.69 mm to (3.37, 27.2), turned to 0 degrees
- moved C11 2.61 mm to (19.3, 13.3)
- moved IC2 2.13 mm to (15.7, 15.4)
- moved RF1 2.10 mm to (33.0, 2.10)
- moved C13 1.92 mm to (12.8, 16.6)
- moved C8 1.92 mm to (10.3, 15.1)
- moved JP1 1.10 mm to (27.1, 6.09)
- moved R9 1.09 mm to (20.9, 6.94)
- moved D1 0.39 mm to (12.4, 20.6)
- moved C12 0.34 mm to (17.1, 9.10)
- moved R13 0.27 mm to (7.46, 9.08), turned to 90 degrees
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Routing:
- net RF_DATA: track 0.00 -> 14.0 mm
- net RST: track 15.8 -> 27.1 mm
- net GND: track 110.2 -> 104.2 mm, vias 4 -> 3
- net BTN1: track 10.9 -> 8.48 mm
- net +5V: track 25.3 -> 27.5 mm
- net SWIM: track 19.2 -> 20.8 mm
- added copper zone on layer 1, net GND

Commit message: PCB work
Parts:
- C4: device resistor:C0805K -> resistor:C0603K
- moved R10 5.72 mm to (3.98, 21.5), flipped to the bottom, turned to 180 degrees
- moved R13 3.26 mm to (6.40, 5.99), turned to 270 degrees
- moved C1 2.50 mm to (17.9, 3.61)
- moved C2 2.50 mm to (15.8, 3.37)
- moved C5 2.32 mm to (17.5, 19.6)
- moved R5 2.24 mm to (16.9, 24.9), turned to 0 degrees
- moved L1 2.20 mm to (7.11, 27.2)
- moved C13 2.05 mm to (11.4, 15.1)
- moved D1 1.84 mm to (10.7, 19.9)
- moved IC2 1.57 mm to (14.1, 15.2)
- moved C4 1.55 mm to (15.2, 26.9), flipped to the bottom, turned to 0 degrees
- moved R7 1.33 mm to (19.8, 24.2)
- moved C8 1.20 mm to (9.13, 15.1)
- moved IC1 1.17 mm to (15.8, 28.8)
- moved C6 1.04 mm to (4.27, 15.7)
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Routing:
- net GND: track 104.2 -> 158.3 mm
- net +3V3: track 48.2 -> 68.3 mm, vias 4 -> 5
- net N$6: track 11.8 -> 6.83 mm, vias 0 -> 20
- net +5V: track 27.5 -> 23.8 mm, vias 0 -> 1
- net BTN1: track 8.48 -> 11.2 mm
- net N$3: track 15.6 -> 13.2 mm
- net N$5: track 3.81 -> 2.30 mm, vias 0 -> 1
- net N$9: track 17.1 -> 16.4 mm
- net N$4: track 7.06 -> 7.61 mm
- net N$1: track 12.8 -> 12.2 mm
- added copper zone on layer 16, net GND
- added copper zone on layer 16, net N$6

Commit message: PCB work
Parts:
- moved LED1 1.81 mm to (43.9, 11.9)
- moved R3 0.80 mm to (38.9, 11.9)
- moved C10 0.80 mm to (44.0, 7.56)
- moved C7 0.80 mm to (36.2, 2.99)
- moved C9 0.80 mm to (42.0, 7.58)
- moved IC3 0.80 mm to (36.7, 8.24)
- moved R2 0.80 mm to (39.8, 3.04)
- moved JP1 0.50 mm to (26.6, 6.09)
- moved R12 0.50 mm to (18.5, 6.80)
- moved R9 0.50 mm to (20.4, 6.11)
- moved S1 0.50 mm to (11.9, 9.09)
- moved C12 0.50 mm to (16.6, 9.10)
- moved R13 0.20 mm to (6.20, 5.99)
Routing:
- net +3V3: track 68.3 -> 66.3 mm
- net GND: track 158.3 -> 159.7 mm
- net N$11: track 9.34 -> 8.54 mm
- net LED_TX_ERR2: track 9.71 -> 10.5 mm

Commit message: PCB work
Routing:
- net +3V3: track 66.3 -> 71.7 mm
Changed lines of the file:
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@@
 <board>
 <plain>
-<wire x1="3.85" y1="43" x2="3.85" y2="39.3" width="0" layer="20"/>
-<wire x1="3.85" y1="39.3" x2="0.25" y2="35.7" width="0" layer="20" curve="-90"/>
+<wire x1="3.85" y1="43" x2="3.85" y2="39.3" width="0.1" layer="20"/>
+<wire x1="3.85" y1="39.3" x2="0.25" y2="35.7" width="0.1" layer="20" curve="-90"/>
 <wire x1="0.25" y1="35.7" x2="0" y2="35.7" width="0" layer="20"/>
-<wire x1="0" y1="35.7" x2="0" y2="1" width="0" layer="20"/>
-<wire x1="0" y1="1" x2="46.15" y2="1" width="0" layer="20"/>
+<wire x1="0" y1="35.7" x2="0" y2="1" width="0.1" layer="20"/>
+<wire x1="0" y1="1" x2="46.15" y2="1" width="0.1" layer="20"/>
 <wire x1="46.15" y1="1" x2="46.15" y2="4.7" width="0" layer="20"/>
-<wire x1="46.15" y1="4.7" x2="49.75" y2="8.3" width="0" layer="20" curve="-90"/>
+<wire x1="46.15" y1="4.7" x2="49.75" y2="8.3" width="0.1" layer="20" curve="-90"/>
 <wire x1="49.75" y1="8.3" x2="50" y2="8.3" width="0" layer="20"/>
-<wire x1="50" y1="8.3" x2="50" y2="43" width="0" layer="20"/>
-<wire x1="50" y1="43" x2="3.85" y2="43" width="0" layer="20"/>
+<wire x1="50" y1="8.3" x2="50" y2="43" width="0.1" layer="20"/>
+<wire x1="50" y1="43" x2="3.85" y2="43" width="0.1" layer="20"/>
 <text x="24.648" y="7.9" size="0.8128" layer="21" font="vector" ratio="20">SW</text>
 <text x="29.725" y="7.9" size="0.8128" layer="21" font="vector" ratio="20">RS</text>
@@
 <wire x1="20.399" y1="5.262" x2="19.137" y2="4" width="0.4064" layer="1"/>
 <wire x1="19.137" y1="4" x2="14.083" y2="4" width="0.4064" layer="1"/>
-<wire x1="9.14" y1="2.626" x2="6.203" y2="5.144" width="0" layer="19" extent="1-1"/>
+<wire x1="6.203" y1="5.144" x2="8.002" y2="5.144" width="0.4064" layer="16"/>
+<wire x1="8.002" y1="5.144" x2="9.156" y2="3.99" width="0.4064" layer="16"/>
+<wire x1="9.156" y1="3.99" x2="9.156" y2="2.131" width="0.4064" layer="16"/>
+<wire x1="9.156" y1="2.131" x2="9.127" y2="2.102" width="0.4064" layer="16"/>
 </signal>
 <signal name="N$2">
