File: Remote Switch v3/ReceiverController/receiver.brd (EAGLE design)
At the start: 50 x 42 mm, 38 parts, among them IC1 LNK304, IC2 MCP1703CB, IC3 STM8L101F2, J1 POWER_CONN_4, T1 BT136

Commit message: PCB work for Remote Switch
Parts:
- IC3: device componente_RFSwitch:TSSOP20 -> comp_RFSwitch_v3:TSSOP20
- moved R1 0.59 mm to (20.1, 40.4), flipped to the top
- moved J1 0.50 mm to (36.6, 39.0), flipped to the top
- flipped C3 to the top
- flipped S1 to the bottom
- renumbered OK1 to OC1
Connections:
- net L: now also J1.4, R1.1; no longer J1.1, R1.2
- net LOAD: now also J1.1; no longer J1.4
- net N$10: now also R1.2; no longer R1.1
Routing:
- net N: track 16.9 -> 11.5 mm
- net L: track 9.01 -> 4.60 mm
- net GND: track 159.7 -> 158.8 mm
- net N$10: track 7.53 -> 8.12 mm
Other:
- board text added: "L"
- board text added: "LOAD"
- board text added: "N"
