File: Remote Switch v3/ReceiverController/receiver.sch (EAGLE design)
At the start: 40 parts, among them IC1 LNK304, IC2 MCP1703CB, IC3 STM8L101F2, J1 POWER_CONN_4, T1 BT136

Commit message: PCB work
Parts:
- added C13: 100n, resistor:C-EUC0603K
Connections:
- removed net N$19: B1.AC1, R1.1
- new net N$10: B1.AC2, R1.1
- net +5V: now also C13.1
- net GND: now also C13.2
- net N: now also B1.AC1; no longer B1.AC2
Other:
- moved on the sheet: C11, IC2, R1
Changed lines of the file:
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@@
 <part name="GND1" library="supply" deviceset="GND" device=""/>
 <part name="R12" library="resistor" deviceset="R-EU_" device="R0603" value="47"/>
+<part name="C13" library="resistor" deviceset="C-EU" device="C0603K" value="100n"/>
+<part name="GND17" library="supply" deviceset="GND" device=""/>
 </parts>
 <sheets>
@@
 <instance part="GND15" gate="1" x="182.88" y="157.48" rot="R270"/>
 <instance part="LED1" gate="G$1" x="53.34" y="162.56" rot="R270"/>
-<instance part="R1" gate="G$1" x="25.4" y="43.18" rot="R180"/>
+<instance part="R1" gate="G$1" x="25.4" y="33.02" rot="R180"/>
 <instance part="C10" gate="G$1" x="160.02" y="142.24"/>
 <instance part="IC1" gate="G$1" x="73.66" y="45.72"/>
 <instance part="GND8" gate="1" x="132.08" y="40.64"/>
 <instance part="GND5" gate="1" x="50.8" y="27.94"/>
-<instance part="+3V34" gate="G$1" x="180.34" y="60.96"/>
+<instance part="+3V34" gate="G$1" x="187.96" y="60.96"/>
 <instance part="D2" gate="G$1" x="127" y="48.26" rot="R90"/>
 <instance part="L1" gate="G$1" x="116.84" y="53.34" rot="R90"/>
@@
 <instance part="R3" gate="G$1" x="63.5" y="134.62"/>
 <instance part="GND6" gate="1" x="66.04" y="121.92"/>
-<instance part="IC2" gate="G$1" x="167.64" y="53.34"/>
-<instance part="C11" gate="G$1" x="180.34" y="50.8"/>
-<instance part="GND14" gate="1" x="180.34" y="43.18"/>
+<instance part="IC2" gate="G$1" x="175.26" y="53.34"/>
+<instance part="C11" gate="G$1" x="187.96" y="50.8"/>
+<instance part="GND14" gate="1" x="187.96" y="43.18"/>
 <instance part="C8" gate="G$1" x="149.86" y="50.8"/>
-<instance part="GND13" gate="1" x="167.64" y="43.18"/>
+<instance part="GND13" gate="1" x="175.26" y="43.18"/>
 <instance part="GND10" gate="1" x="149.86" y="43.18"/>
 <instance part="RF1" gate="G$1" x="45.72" y="93.98"/>
@@
 <instance part="GND1" gate="1" x="15.24" y="83.82"/>
 <instance part="R12" gate="G$1" x="220.98" y="109.22"/>
+<instance part="C13" gate="G$1" x="157.48" y="50.8"/>
+<instance part="GND17" gate="1" x="157.48" y="43.18"/>
 </instances>
 <busses>
@@
 <junction x="238.76" y="134.62"/>
 <junction x="241.3" y="134.62"/>
+</segment>
+<segment>
+<pinref part="C13" gate="G$1" pin="2"/>
+<pinref part="GND17" gate="1" pin="GND"/>
 </segment>
 </net>
@@
 <pinref part="IC2" gate="G$1" pin="VO"/>
 <pinref part="C11" gate="G$1" pin="1"/>
-<wire x1="177.8" y1="53.34" x2="180.34" y2="53.34" width="0.1524" layer="91"/>
+<wire x1="185.42" y1="53.34" x2="187.96" y2="53.34" width="0.1524" layer="91"/>
 <pinref part="+3V34" gate="G$1" pin="+3V3"/>
-<wire x1="180.34" y1="53.34" x2="180.34" y2="58.42" width="0.1524" layer="91"/>
-<junction x="180.34" y="53.34"/>
+<wire x1="187.96" y1="53.34" x2="187.96" y2="58.42" width="0.1524" layer="91"/>
+<junction x="187.96" y="53.34"/>
 </segment>
 <segment>
@@
 </segment>
 <segment>
-<wire x1="38.1" y1="33.02" x2="12.7" y2="33.02" width="0.1524" layer="91"/>
-<label x="12.7" y="33.02" size="1.778" layer="95"/>
-<pinref part="B1" gate="G$1" pin="AC2"/>
+<pinref part="B1" gate="G$1" pin="AC1"/>
+<wire x1="38.1" y1="43.18" x2="12.7" y2="43.18" width="0.1524" layer="91"/>
+<label x="12.7" y="43.18" size="1.778" layer="95"/>
 </segment>
 </net>
@@
 </segment>
 </net>
-<net name="N$19" class="0">
-<segment>
-<pinref part="R1" gate="G$1" pin="1"/>
-<pinref part="B1" gate="G$1" pin="AC1"/>
-<wire x1="30.48" y1="43.18" x2="38.1" y2="43.18" width="0.1524" layer="91"/>
-</segment>
-</net>
 <net name="L" class="0">
 <segment>
@@
 <segment>
 <pinref part="R1" gate="G$1" pin="2"/>
-<wire x1="20.32" y1="43.18" x2="12.7" y2="43.18" width="0.1524" layer="91"/>
-<label x="12.7" y="43.18" size="1.778" layer="95"/>
+<wire x1="20.32" y1="33.02" x2="12.7" y2="33.02" width="0.1524" layer="91"/>
+<label x="12.7" y="33.02" size="1.778" layer="95"/>
 </segment>
 <segment>
@@
 <junction x="132.08" y="53.34"/>
 <pinref part="IC2" gate="G$1" pin="VI"/>
-<wire x1="157.48" y1="53.34" x2="149.86" y2="53.34" width="0.1524" layer="91"/>
+<wire x1="165.1" y1="53.34" x2="157.48" y2="53.34" width="0.1524" layer="91"/>
 <junction x="142.24" y="53.34"/>
 <pinref part="C8" gate="G$1" pin="1"/>
+<wire x1="157.48" y1="53.34" x2="149.86" y2="53.34" width="0.1524" layer="91"/>
 <wire x1="149.86" y1="53.34" x2="142.24" y2="53.34" width="0.1524" layer="91"/>
 <junction x="149.86" y="53.34"/>
 <label x="144.78" y="53.34" size="1.778" layer="95"/>
+<pinref part="C13" gate="G$1" pin="1"/>
+<junction x="157.48" y="53.34"/>
 </segment>
 </net>
@@
 </segment>
 </net>
+<net name="N$10" class="0">
+<segment>
+<pinref part="R1" gate="G$1" pin="1"/>
+<pinref part="B1" gate="G$1" pin="AC2"/>
+<wire x1="30.48" y1="33.02" x2="38.1" y2="33.02" width="0.1524" layer="91"/>
+</segment>
+</net>

Commit message: PCB work
Connections:
- net N$6: now also IC1.S@1, IC1.S@2, IC1.S@3, IC1.S@4; no longer IC1.S1, IC1.S2, IC1.S3, IC1.S4
Changed lines of the file:
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@@
 <pinref part="C4" gate="G$1" pin="2"/>
 <wire x1="76.2" y1="60.96" x2="86.36" y2="60.96" width="0.1524" layer="91"/>
-<pinref part="IC1" gate="G$1" pin="S1"/>
+<pinref part="IC1" gate="G$1" pin="S@1"/>
 <wire x1="86.36" y1="60.96" x2="86.36" y2="53.34" width="0.1524" layer="91"/>
-<pinref part="IC1" gate="G$1" pin="S2"/>
+<pinref part="IC1" gate="G$1" pin="S@2"/>
 <wire x1="86.36" y1="53.34" x2="86.36" y2="48.26" width="0.1524" layer="91"/>
 <junction x="86.36" y="53.34"/>
-<pinref part="IC1" gate="G$1" pin="S3"/>
+<pinref part="IC1" gate="G$1" pin="S@3"/>
 <wire x1="86.36" y1="48.26" x2="86.36" y2="43.18" width="0.1524" layer="91"/>
 <junction x="86.36" y="48.26"/>
-<pinref part="IC1" gate="G$1" pin="S4"/>
+<pinref part="IC1" gate="G$1" pin="S@4"/>
 <wire x1="86.36" y1="43.18" x2="86.36" y2="38.1" width="0.1524" layer="91"/>
 <junction x="86.36" y="43.18"/>

Commit message: PCB work
Parts:
- removed SIG_1, SIG_2, SIG_3, SIG_4: CON_PAD, componente_RFSwitch:CON_PAD
- added JP1: (no value), pinhead:PINHD-1X4
Connections:
- net +3V3: now also JP1.1; no longer SIG_1.P$1
- net GND: now also JP1.3; no longer SIG_3.P$1
- net RST: now also JP1.4; no longer SIG_4.P$1
- net SWIM: now also JP1.2; no longer SIG_2.P$1
Changed lines of the file:
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@@
 <part name="+3V36" library="supply1" deviceset="+3V3" device=""/>
 <part name="J1" library="CarReceiver" deviceset="POWER_CONN_4" device=""/>
-<part name="SIG_1" library="componente_RFSwitch" deviceset="CON_PAD" device=""/>
-<part name="SIG_2" library="componente_RFSwitch" deviceset="CON_PAD" device=""/>
-<part name="SIG_3" library="componente_RFSwitch" deviceset="CON_PAD" device=""/>
-<part name="SIG_4" library="componente_RFSwitch" deviceset="CON_PAD" device=""/>
 <part name="+3V35" library="supply1" deviceset="+3V3" device=""/>
 <part name="GND15" library="supply" deviceset="GND" device=""/>
@@
 <part name="C13" library="resistor" deviceset="C-EU" device="C0603K" value="100n"/>
 <part name="GND17" library="supply" deviceset="GND" device=""/>
+<part name="JP1" library="pinhead" deviceset="PINHD-1X4" device=""/>
 </parts>
 <sheets>
@@
 <instance part="+3V36" gate="G$1" x="238.76" y="157.48"/>
 <instance part="J1" gate="G$1" x="17.78" y="129.54"/>
-<instance part="SIG_1" gate="G$1" x="187.96" y="162.56"/>
-<instance part="SIG_2" gate="G$1" x="187.96" y="160.02"/>
-<instance part="SIG_3" gate="G$1" x="187.96" y="157.48"/>
-<instance part="SIG_4" gate="G$1" x="187.96" y="154.94"/>
-<instance part="+3V35" gate="G$1" x="187.96" y="167.64"/>
-<instance part="GND15" gate="1" x="182.88" y="157.48" rot="R270"/>
+<instance part="+3V35" gate="G$1" x="208.28" y="172.72"/>
+<instance part="GND15" gate="1" x="205.74" y="157.48" rot="R270"/>
 <instance part="LED1" gate="G$1" x="53.34" y="162.56" rot="R270"/>
 <instance part="R1" gate="G$1" x="25.4" y="33.02" rot="R180"/>
@@
 <instance part="C13" gate="G$1" x="157.48" y="50.8"/>
 <instance part="GND17" gate="1" x="157.48" y="43.18"/>
+<instance part="JP1" gate="A" x="210.82" y="157.48"/>
 </instances>
 <busses>
@@
 </segment>
 <segment>
-<pinref part="SIG_4" gate="G$1" pin="P$1"/>
-<wire x1="187.96" y1="154.94" x2="198.12" y2="154.94" width="0.1524" layer="91"/>
-<label x="190.5" y="154.94" size="1.778" layer="95"/>
+<pinref part="JP1" gate="A" pin="4"/>
+<wire x1="208.28" y1="154.94" x2="195.58" y2="154.94" width="0.1524" layer="91"/>
+<label x="195.58" y="154.94" size="1.778" layer="95"/>
 </segment>
 </net>
@@
 <junction x="152.4" y="137.16"/>
 <pinref part="C10" gate="G$1" pin="2"/>
-</segment>
-<segment>
-<pinref part="SIG_3" gate="G$1" pin="P$1"/>
-<pinref part="GND15" gate="1" pin="GND"/>
-<wire x1="185.42" y1="157.48" x2="187.96" y2="157.48" width="0.1524" layer="91"/>
 </segment>
 <segment>
@@
 <pinref part="C13" gate="G$1" pin="2"/>
 <pinref part="GND17" gate="1" pin="GND"/>
+</segment>
+<segment>
+<pinref part="JP1" gate="A" pin="3"/>
+<pinref part="GND15" gate="1" pin="GND"/>
 </segment>
 </net>
@@
 </segment>
 <segment>
-<pinref part="SIG_2" gate="G$1" pin="P$1"/>
-<wire x1="187.96" y1="160.02" x2="198.12" y2="160.02" width="0.1524" layer="91"/>
-<label x="190.5" y="160.02" size="1.778" layer="95"/>
+<pinref part="JP1" gate="A" pin="2"/>
+<wire x1="208.28" y1="160.02" x2="195.58" y2="160.02" width="0.1524" layer="91"/>
+<label x="195.58" y="160.02" size="1.778" layer="95"/>
 </segment>
 </net>
@@
 </segment>
 <segment>
-<pinref part="SIG_1" gate="G$1" pin="P$1"/>
-<pinref part="+3V35" gate="G$1" pin="+3V3"/>
-<wire x1="187.96" y1="165.1" x2="187.96" y2="162.56" width="0.1524" layer="91"/>
-</segment>
-<segment>
 <pinref part="IC2" gate="G$1" pin="VO"/>
 <pinref part="C11" gate="G$1" pin="1"/>
@@
 <wire x1="25.4" y1="93.98" x2="15.24" y2="93.98" width="0.1524" layer="91"/>
 </segment>
-</net>
+<segment>
+<pinref part="+3V35" gate="G$1" pin="+3V3"/>
+<pinref part="JP1" gate="A" pin="1"/>
+<wire x1="208.28" y1="170.18" x2="208.28" y2="162.56" width="0.1524" layer="91"/>
+</segment>
+</net>

Commit message: PCB work
Parts:
- C4: device resistor:C-EUC0805K -> resistor:C-EUC0603K
Changed lines of the file:
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@@
 <grid distance="0.1" unitdist="inch" unit="inch" style="lines" multiple="1" display="no" altdistance="0.01" altunitdist="inch" altunit="inch"/>
 <layers>
-<layer number="1" name="Top" color="4" fill="1" visible="no" active="no"/>
-<layer number="16" name="Bottom" color="1" fill="1" visible="no" active="no"/>
-<layer number="17" name="Pads" color="2" fill="1" visible="no" active="no"/>
-<layer number="18" name="Vias" color="2" fill="1" visible="no" active="no"/>
-<layer number="19" name="Unrouted" color="6" fill="1" visible="no" active="no"/>
-<layer number="20" name="Dimension" color="15" fill="1" visible="no" active="no"/>
-<layer number="21" name="tPlace" color="7" fill="1" visible="no" active="no"/>
-<layer number="22" name="bPlace" color="7" fill="1" visible="no" active="no"/>
-<layer number="23" name="tOrigins" color="15" fill="1" visible="no" active="no"/>
-<layer number="24" name="bOrigins" color="15" fill="1" visible="no" active="no"/>
-<layer number="25" name="tNames" color="7" fill="1" visible="no" active="no"/>
-<layer number="26" name="bNames" color="7" fill="1" visible="no" active="no"/>
-<layer number="27" name="tValues" color="7" fill="1" visible="no" active="no"/>
-<layer number="28" name="bValues" color="7" fill="1" visible="no" active="no"/>
+<layer number="1" name="Top" color="4" fill="1" visible="yes" active="no"/>
+<layer number="16" name="Bottom" color="1" fill="1" visible="yes" active="no"/>
+<layer number="17" name="Pads" color="2" fill="1" visible="yes" active="no"/>
+<layer number="18" name="Vias" color="2" fill="1" visible="yes" active="no"/>
+<layer number="19" name="Unrouted" color="6" fill="1" visible="yes" active="no"/>
+<layer number="20" name="Dimension" color="15" fill="1" visible="yes" active="no"/>
+<layer number="21" name="tPlace" color="7" fill="1" visible="yes" active="no"/>
+<layer number="22" name="bPlace" color="7" fill="1" visible="yes" active="no"/>
+<layer number="23" name="tOrigins" color="15" fill="1" visible="yes" active="no"/>
+<layer number="24" name="bOrigins" color="15" fill="1" visible="yes" active="no"/>
+<layer number="25" name="tNames" color="7" fill="1" visible="yes" active="no"/>
+<layer number="26" name="bNames" color="7" fill="1" visible="yes" active="no"/>
+<layer number="27" name="tValues" color="7" fill="1" visible="yes" active="no"/>
+<layer number="28" name="bValues" color="7" fill="1" visible="yes" active="no"/>
 <layer number="29" name="tStop" color="7" fill="3" visible="no" active="no"/>
 <layer number="30" name="bStop" color="7" fill="6" visible="no" active="no"/>
@@
 <layer number="35" name="tGlue" color="7" fill="4" visible="no" active="no"/>
 <layer number="36" name="bGlue" color="7" fill="5" visible="no" active="no"/>
-<layer number="37" name="tTest" color="7" fill="1" visible="no" active="no"/>
-<layer number="38" name="bTest" color="7" fill="1" visible="no" active="no"/>
+<layer number="37" name="tTest" color="7" fill="1" visible="yes" active="no"/>
+<layer number="38" name="bTest" color="7" fill="1" visible="yes" active="no"/>
 <layer number="39" name="tKeepout" color="4" fill="11" visible="no" active="no"/>
 <layer number="40" name="bKeepout" color="1" fill="11" visible="no" active="no"/>
@@
 <layer number="44" name="Drills" color="7" fill="1" visible="no" active="no"/>
 <layer number="45" name="Holes" color="7" fill="1" visible="no" active="no"/>
-<layer number="46" name="Milling" color="3" fill="1" visible="no" active="no"/>
-<layer number="47" name="Measures" color="7" fill="1" visible="no" active="no"/>
-<layer number="48" name="Document" color="7" fill="1" visible="no" active="no"/>
-<layer number="49" name="Reference" color="7" fill="1" visible="no" active="no"/>
-<layer number="50" name="dxf" color="7" fill="1" visible="no" active="no"/>
-<layer number="51" name="tDocu" color="7" fill="1" visible="no" active="no"/>
-<layer number="52" name="bDocu" color="7" fill="1" visible="no" active="no"/>
-<layer number="53" name="tGND_GNDA" color="7" fill="9" visible="no" active="no"/>
-<layer number="54" name="bGND_GNDA" color="1" fill="9" visible="no" active="no"/>
-<layer number="56" name="wert" color="7" fill="1" visible="no" active="no"/>
+<layer number="46" name="Milling" color="3" fill="1" visible="yes" active="no"/>
+<layer number="47" name="Measures" color="7" fill="1" visible="yes" active="no"/>
+<layer number="48" name="Document" color="7" fill="1" visible="yes" active="no"/>
+<layer number="49" name="Reference" color="7" fill="1" visible="yes" active="no"/>
+<layer number="50" name="dxf" color="7" fill="1" visible="yes" active="no"/>
+<layer number="51" name="tDocu" color="7" fill="1" visible="yes" active="no"/>
+<layer number="52" name="bDocu" color="7" fill="1" visible="yes" active="no"/>
+<layer number="53" name="tGND_GNDA" color="7" fill="9" visible="yes" active="no"/>
+<layer number="54" name="bGND_GNDA" color="1" fill="9" visible="yes" active="no"/>
+<layer number="56" name="wert" color="7" fill="1" visible="yes" active="no"/>
 <layer number="90" name="Modules" color="5" fill="1" visible="no" active="no"/>
 <layer number="91" name="Nets" color="2" fill="1" visible="yes" active="yes"/>
@@
 <part name="B1" library="rectifier" deviceset="B*S" device="" technology="05"/>
 <part name="C3" library="resistor" deviceset="CPOL-EU" device="E5-10.5" value="4.7u"/>
-<part name="C4" library="resistor" deviceset="C-EU" device="C0805K" value="100n"/>
+<part name="C4" library="resistor" deviceset="C-EU" device="C0603K" value="100n"/>
 <part name="C6" library="resistor" deviceset="CPOL-EU" device="D" value="100u"/>
 <part name="+3V33" library="supply1" deviceset="+3V3" device=""/>
