File: Remote Switch v3/ReceiverController/receiver.sch (EAGLE design)
At the start: 38 parts, among them IC1 LNK304, IC2 MCP1703CB, IC3 STM8L101F2, J1 POWER_CONN_4, T1 BT136

Commit message: PCB work for Remote Switch
Parts:
- IC3: device componente_RFSwitch:STM8L101F2 -> comp_RFSwitch_v3:STM8L101F2
- renumbered OK1 to OC1
Connections:
- net L: now also J1.P$4, R1.1; no longer J1.P$1, R1.2
- net LOAD: now also J1.P$1; no longer J1.P$4
- net N$10: now also R1.2; no longer R1.1
Other:
- moved on the sheet: R1
Changed lines of the file:
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@@
 <grid distance="0.1" unitdist="inch" unit="inch" style="lines" multiple="1" display="no" altdistance="0.01" altunitdist="inch" altunit="inch"/>
 <layers>
-<layer number="1" name="Top" color="4" fill="1" visible="yes" active="no"/>
-<layer number="16" name="Bottom" color="1" fill="1" visible="yes" active="no"/>
-<layer number="17" name="Pads" color="2" fill="1" visible="yes" active="no"/>
-<layer number="18" name="Vias" color="2" fill="1" visible="yes" active="no"/>
-<layer number="19" name="Unrouted" color="6" fill="1" visible="yes" active="no"/>
-<layer number="20" name="Dimension" color="15" fill="1" visible="yes" active="no"/>
-<layer number="21" name="tPlace" color="7" fill="1" visible="yes" active="no"/>
-<layer number="22" name="bPlace" color="7" fill="1" visible="yes" active="no"/>
-<layer number="23" name="tOrigins" color="15" fill="1" visible="yes" active="no"/>
-<layer number="24" name="bOrigins" color="15" fill="1" visible="yes" active="no"/>
-<layer number="25" name="tNames" color="7" fill="1" visible="yes" active="no"/>
-<layer number="26" name="bNames" color="7" fill="1" visible="yes" active="no"/>
-<layer number="27" name="tValues" color="7" fill="1" visible="yes" active="no"/>
-<layer number="28" name="bValues" color="7" fill="1" visible="yes" active="no"/>
+<layer number="1" name="Top" color="4" fill="1" visible="no" active="no"/>
+<layer number="16" name="Bottom" color="1" fill="1" visible="no" active="no"/>
+<layer number="17" name="Pads" color="2" fill="1" visible="no" active="no"/>
+<layer number="18" name="Vias" color="2" fill="1" visible="no" active="no"/>
+<layer number="19" name="Unrouted" color="6" fill="1" visible="no" active="no"/>
+<layer number="20" name="Dimension" color="15" fill="1" visible="no" active="no"/>
+<layer number="21" name="tPlace" color="7" fill="1" visible="no" active="no"/>
+<layer number="22" name="bPlace" color="7" fill="1" visible="no" active="no"/>
+<layer number="23" name="tOrigins" color="15" fill="1" visible="no" active="no"/>
+<layer number="24" name="bOrigins" color="15" fill="1" visible="no" active="no"/>
+<layer number="25" name="tNames" color="7" fill="1" visible="no" active="no"/>
+<layer number="26" name="bNames" color="7" fill="1" visible="no" active="no"/>
+<layer number="27" name="tValues" color="7" fill="1" visible="no" active="no"/>
+<layer number="28" name="bValues" color="7" fill="1" visible="no" active="no"/>
 <layer number="29" name="tStop" color="7" fill="3" visible="no" active="no"/>
 <layer number="30" name="bStop" color="7" fill="6" visible="no" active="no"/>
@@
 <layer number="35" name="tGlue" color="7" fill="4" visible="no" active="no"/>
 <layer number="36" name="bGlue" color="7" fill="5" visible="no" active="no"/>
-<layer number="37" name="tTest" color="7" fill="1" visible="yes" active="no"/>
-<layer number="38" name="bTest" color="7" fill="1" visible="yes" active="no"/>
+<layer number="37" name="tTest" color="7" fill="1" visible="no" active="no"/>
+<layer number="38" name="bTest" color="7" fill="1" visible="no" active="no"/>
 <layer number="39" name="tKeepout" color="4" fill="11" visible="no" active="no"/>
 <layer number="40" name="bKeepout" color="1" fill="11" visible="no" active="no"/>
@@
 <layer number="44" name="Drills" color="7" fill="1" visible="no" active="no"/>
 <layer number="45" name="Holes" color="7" fill="1" visible="no" active="no"/>
-<layer number="46" name="Milling" color="3" fill="1" visible="yes" active="no"/>
-<layer number="47" name="Measures" color="7" fill="1" visible="yes" active="no"/>
-<layer number="48" name="Document" color="7" fill="1" visible="yes" active="no"/>
-<layer number="49" name="Reference" color="7" fill="1" visible="yes" active="no"/>
-<layer number="50" name="dxf" color="7" fill="1" visible="yes" active="no"/>
-<layer number="51" name="tDocu" color="7" fill="1" visible="yes" active="no"/>
-<layer number="52" name="bDocu" color="7" fill="1" visible="yes" active="no"/>
-<layer number="53" name="tGND_GNDA" color="7" fill="9" visible="yes" active="no"/>
-<layer number="54" name="bGND_GNDA" color="1" fill="9" visible="yes" active="no"/>
-<layer number="56" name="wert" color="7" fill="1" visible="yes" active="no"/>
+<layer number="46" name="Milling" color="3" fill="1" visible="no" active="no"/>
+<layer number="47" name="Measures" color="7" fill="1" visible="no" active="no"/>
+<layer number="48" name="Document" color="7" fill="1" visible="no" active="no"/>
+<layer number="49" name="Reference" color="7" fill="1" visible="no" active="no"/>
+<layer number="50" name="dxf" color="7" fill="1" visible="no" active="no"/>
+<layer number="51" name="tDocu" color="7" fill="1" visible="no" active="no"/>
+<layer number="52" name="bDocu" color="7" fill="1" visible="no" active="no"/>
+<layer number="53" name="tGND_GNDA" color="7" fill="9" visible="no" active="no"/>
+<layer number="54" name="bGND_GNDA" color="1" fill="9" visible="no" active="no"/>
+<layer number="56" name="wert" color="7" fill="1" visible="no" active="no"/>
 <layer number="90" name="Modules" color="5" fill="1" visible="no" active="no"/>
 <layer number="91" name="Nets" color="2" fill="1" visible="yes" active="yes"/>
@@
 </classes>
 <parts>
-<part name="IC3" library="componente_RFSwitch" deviceset="STM8L101F2" device=""/>
+<part name="IC3" library="comp_RFSwitch_v3" deviceset="STM8L101F2" device=""/>
 <part name="R9" library="resistor" deviceset="R-EU_" device="R0603" value="10k"/>
 <part name="C7" library="resistor" deviceset="C-EU" device="C0603K" value="100n"/>
@@
 <part name="R5" library="resistor" deviceset="R-EU_" device="R0603" value="1k"/>
 <part name="T1" library="triac" deviceset="BT136" device=""/>
-<part name="OK1" library="optocoupler" deviceset="MOC30*M" device="" technology="23" value="MOC3063M"/>
+<part name="OC1" library="optocoupler" deviceset="MOC30*M" device="" technology="23" value="MOC3063M"/>
 <part name="R6" library="resistor" deviceset="R-EU_" device="R0805" value="360"/>
 <part name="R4" library="resistor" deviceset="R-EU_" device="R0805" value="360"/>
@@
 <instance part="GND15" gate="1" x="205.74" y="157.48" rot="R270"/>
 <instance part="LED1" gate="G$1" x="53.34" y="162.56" rot="R270"/>
-<instance part="R1" gate="G$1" x="25.4" y="33.02" rot="R180"/>
+<instance part="R1" gate="G$1" x="25.4" y="33.02"/>
 <instance part="C10" gate="G$1" x="160.02" y="142.24"/>
 <instance part="IC1" gate="G$1" x="73.66" y="45.72"/>
@@
 <instance part="R5" gate="G$1" x="91.44" y="63.5" rot="R90"/>
 <instance part="T1" gate="-1" x="99.06" y="127"/>
-<instance part="OK1" gate="-1" x="78.74" y="129.54"/>
+<instance part="OC1" gate="-1" x="78.74" y="129.54"/>
 <instance part="R6" gate="G$1" x="93.98" y="134.62"/>
 <instance part="R4" gate="G$1" x="88.9" y="119.38" rot="R90"/>
@@
 </segment>
 <segment>
-<pinref part="OK1" gate="-1" pin="C"/>
+<pinref part="OC1" gate="-1" pin="C"/>
 <pinref part="GND6" gate="1" pin="GND"/>
 <wire x1="66.04" y1="124.46" x2="68.58" y2="124.46" width="0.1524" layer="91"/>
@@
 <net name="L" class="0">
 <segment>
-<pinref part="J1" gate="G$1" pin="P$1"/>
-<label x="25.4" y="137.16" size="1.778" layer="95"/>
-<wire x1="22.86" y1="137.16" x2="27.94" y2="137.16" width="0.1524" layer="91"/>
-</segment>
-<segment>
-<pinref part="R1" gate="G$1" pin="2"/>
-<wire x1="20.32" y1="33.02" x2="12.7" y2="33.02" width="0.1524" layer="91"/>
-<label x="12.7" y="33.02" size="1.778" layer="95"/>
-</segment>
-<segment>
 <pinref part="R4" gate="G$1" pin="1"/>
 <wire x1="88.9" y1="114.3" x2="99.06" y2="114.3" width="0.1524" layer="91"/>
@@
 <junction x="99.06" y="114.3"/>
 <label x="101.6" y="114.3" size="1.778" layer="95"/>
+</segment>
+<segment>
+<pinref part="R1" gate="G$1" pin="1"/>
+<wire x1="20.32" y1="33.02" x2="12.7" y2="33.02" width="0.1524" layer="91"/>
+<label x="12.7" y="33.02" size="1.778" layer="95"/>
+</segment>
+<segment>
+<pinref part="J1" gate="G$1" pin="P$4"/>
+<wire x1="22.86" y1="121.92" x2="27.94" y2="121.92" width="0.1524" layer="91"/>
+<label x="25.4" y="121.92" size="1.778" layer="95"/>
 </segment>
 </net>
@@
 <net name="N$7" class="0">
 <segment>
-<pinref part="OK1" gate="-1" pin="A2"/>
+<pinref part="OC1" gate="-1" pin="A2"/>
 <pinref part="R6" gate="G$1" pin="1"/>
 </segment>
@@
 <pinref part="T1" gate="-1" pin="G"/>
 <wire x1="93.98" y1="127" x2="88.9" y2="127" width="0.1524" layer="91"/>
-<pinref part="OK1" gate="-1" pin="A1"/>
+<pinref part="OC1" gate="-1" pin="A1"/>
 <wire x1="88.9" y1="127" x2="88.9" y2="124.46" width="0.1524" layer="91"/>
 <pinref part="R4" gate="G$1" pin="2"/>
@@
 <net name="N$11" class="0">
 <segment>
-<pinref part="OK1" gate="-1" pin="A"/>
+<pinref part="OC1" gate="-1" pin="A"/>
 <pinref part="R3" gate="G$1" pin="2"/>
 </segment>
@@
 <net name="LOAD" class="0">
 <segment>
-<pinref part="J1" gate="G$1" pin="P$4"/>
-<wire x1="22.86" y1="121.92" x2="27.94" y2="121.92" width="0.1524" layer="91"/>
-<label x="25.4" y="121.92" size="1.778" layer="95"/>
-</segment>
-<segment>
 <pinref part="R6" gate="G$1" pin="2"/>
 <pinref part="T1" gate="-1" pin="A2"/>
@@
 <label x="101.6" y="134.62" size="1.778" layer="95"/>
 </segment>
+<segment>
+<pinref part="J1" gate="G$1" pin="P$1"/>
+<label x="25.4" y="137.16" size="1.778" layer="95"/>
+<wire x1="22.86" y1="137.16" x2="27.94" y2="137.16" width="0.1524" layer="91"/>
+</segment>
 </net>
 <net name="N$9" class="0">
@@
 <net name="N$10" class="0">
 <segment>
-<pinref part="R1" gate="G$1" pin="1"/>
+<pinref part="R1" gate="G$1" pin="2"/>
 <pinref part="B1" gate="G$1" pin="AC2"/>
 <wire x1="30.48" y1="33.02" x2="38.1" y2="33.02" width="0.1524" layer="91"/>
