File: Remote Switch v3/EmitterSwitch/emitter.sch (EAGLE design)
At the start: 29 parts, among them IC2 STM8L101F2, Q1 MMBT3906LT1SMD

Commit message: PCB work
Parts:
- removed R10: 1K, resistor:R-EU_R0603
- removed R11, R12, R7, R8, R9: 10k, resistor:R-EU_R0603
- removed SIG_+3V1, SIG_GND, SIG_RST, SIG_SWIM: CON_PAD, componente_RFSwitch:CON_PAD
- removed U$1: MINI_NRF24L01+, comp_RFSwitch_v2:MINI_NRF24L01+
- removed U$2: CR2032_HOLDER_BC-2003, comp_RFSwitch_v2:CR2032_HOLDER_BC-2003
- added IC1: STM8L101F2, comp_RFSwitch_v2:STM8L101F2
- added JP1: (no value), pinhead:PINHD-1X4
- added R2: 10k, resistor:R-EU_R0603
- added S1: DTSM-3, switch-tact:DTSM-3
- B1: value DTSM-3 -> (none); device switch-tact:DTSM-3 -> comp_RFSwitch_v2:CR2032_HOLDER_BC-2003
- IC2: value STM8L101F2 -> RFM85W; device comp_RFSwitch_v2:STM8L101F2 -> comp_RFSwitch_v3:RFM85W
- R5, R6: value 10k -> 1K
- renumbered B2 to S2, ERR/TX to LED1
Connections:
- removed net N$4: Q1.C, U$1.1
- removed net NRF_CE: IC2.PB3, R5.2, U$1.4
- removed net NRF_CSN: IC2.PB2, R4.1, U$1.3
- removed net NRF_IRQ: IC2.PC2, R7.1, U$1.8
- removed net NRF_MISO: IC2.PB7, R9.2, U$1.7
- removed net NRF_MOSI: IC2.PB6, R11.2, U$1.6
- removed net NRF_ON: IC2.PB1, R10.1
- removed net NRF_SCK: IC2.PB5, R12.2, U$1.5
- new net N$2: IC2.3, Q1.C
- new net RFM85_DATA: IC2.2, R6.2
- new net RFM85_ON: IC1.PB1, R5.1
- new net UC_RFM85_DATA: IC1.PB3, R6.1
- net +3V0: now also B1.+, IC1.VDD, JP1.1, R2.2; no longer IC2.VDD, R6.2, R7.2, R8.2, SIG_+3V1.P$1, U$2.+
- net BTN1: now also IC1.PC4, R3.1, S1.2; no longer B1.2, IC2.PB0, R6.1
- net BTN2: now also IC1.PB0, R4.1; no longer IC2.PD0, R8.1
- net GND: now also B1.-, IC1.VSS, IC2.1, JP1.3, S1.1; no longer B1.1, IC2.VSS, R11.1, R12.1, R5.1, R9.1, SIG_GND.P$1, U$1.2, U$2.-
- net LED_ERR_TX1: now also IC1.PD0; no longer IC2.PC3
- net LED_ERR_TX2: now also IC1.PC3; no longer IC2.PC4
- net N$8: now also R5.2; no longer R10.2
- net RST: now also IC1.NRST/PA1, JP1.4, R2.1; no longer IC2.NRST/PA1, R3.1, SIG_RST.P$1
- net SWIM: now also IC1.PA0, JP1.2; no longer IC2.PA0, SIG_SWIM.P$1
Other:
- moved on the sheet: R3, R4, R5, R6

Commit message: PCB work for Remote Switch
Connections:
- net BTN1: now also IC1.PC2; no longer IC1.PC4
- net BTN2: now also IC1.PC1; no longer IC1.PB0
- net LED_ERR_TX1: now also IC1.PA3; no longer IC1.PD0
- net LED_ERR_TX2: now also IC1.PA2; no longer IC1.PC3
- net RFM85_ON: now also IC1.PC3; no longer IC1.PB1
Changed lines of the file:
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@@
 </segment>
 <segment>
-<wire x1="86.36" y1="91.44" x2="76.2" y2="91.44" width="0.1524" layer="91"/>
-<label x="76.2" y="91.44" size="1.778" layer="95"/>
-<pinref part="IC1" gate="G$1" pin="PC4"/>
+<pinref part="IC1" gate="G$1" pin="PC2"/>
+<wire x1="134.62" y1="109.22" x2="142.24" y2="109.22" width="0.1524" layer="91"/>
+<label x="137.16" y="109.22" size="1.778" layer="95"/>
 </segment>
 </net>
@@
 </segment>
 <segment>
-<pinref part="IC1" gate="G$1" pin="PB0"/>
-<wire x1="86.36" y1="86.36" x2="76.2" y2="86.36" width="0.1524" layer="91"/>
-<label x="76.2" y="86.36" size="1.778" layer="95"/>
+<pinref part="IC1" gate="G$1" pin="PC1"/>
+<wire x1="134.62" y1="106.68" x2="142.24" y2="106.68" width="0.1524" layer="91"/>
+<label x="137.16" y="106.68" size="1.778" layer="95"/>
 </segment>
 </net>
@@
 </segment>
 <segment>
-<pinref part="IC1" gate="G$1" pin="PC3"/>
-<wire x1="86.36" y1="93.98" x2="68.58" y2="93.98" width="0.1524" layer="91"/>
-<label x="68.58" y="93.98" size="1.778" layer="95"/>
+<pinref part="IC1" gate="G$1" pin="PA2"/>
+<wire x1="86.36" y1="101.6" x2="68.58" y2="101.6" width="0.1524" layer="91"/>
+<label x="68.58" y="101.6" size="1.778" layer="95"/>
 </segment>
 </net>
@@
 </segment>
 <segment>
-<pinref part="IC1" gate="G$1" pin="PD0"/>
-<wire x1="86.36" y1="88.9" x2="68.58" y2="88.9" width="0.1524" layer="91"/>
-<label x="68.58" y="88.9" size="1.778" layer="95"/>
+<pinref part="IC1" gate="G$1" pin="PA3"/>
+<wire x1="86.36" y1="99.06" x2="68.58" y2="99.06" width="0.1524" layer="91"/>
+<label x="68.58" y="99.06" size="1.778" layer="95"/>
 </segment>
 </net>
@@
 </segment>
 <segment>
-<pinref part="IC1" gate="G$1" pin="PB1"/>
-<wire x1="134.62" y1="86.36" x2="152.4" y2="86.36" width="0.1524" layer="91"/>
-<label x="137.16" y="86.36" size="1.778" layer="95"/>
+<pinref part="IC1" gate="G$1" pin="PC3"/>
+<wire x1="86.36" y1="93.98" x2="71.12" y2="93.98" width="0.1524" layer="91"/>
+<label x="71.12" y="93.98" size="1.778" layer="95"/>
 </segment>
 </net>
