File: Remote Switch v3.1/ReceiverController/receiver.sch (EAGLE design)
At the start: 38 parts, among them IC1 LNK304, IC2 MCP1703CB, IC3 STM8L101F2, J1 POWER_CONN_4, T1 BT136

Commit message: PCB work - almost complete
Parts:
- C1, C11, C12, C8: device resistor:C-EUC0805K -> resistor:C-EUC1206
- C3: device resistor:CPOL-EUE5-10.5 -> comp_RFSwitch_v3:C-POL-EUE5-10,5
- D1: value S1G-DIO -> US1G-DIO; device comp_RFSwitch_v3:S1G-DIO -> comp_RFSwitch_v3:US1G-DIO
- D2: value US1G-DIO -> S1G-DIO; device comp_RFSwitch_v3:US1G-DIO -> comp_RFSwitch_v3:S1G-DIO
- JP1: device pinhead:PINHD-1X4 -> comp_RFSwitch_v3:CON_1X4PIN_2.54MM_SMD
- R1: value 10 -> 4R7; device resistor:R-EU_0309/10 -> comp_RFSwitch_v3:R_R2512_LARGER_PADS
- R4, R6: device resistor:R-EU_R0805 -> resistor:R-EU_R0603
- renumbered BTN1 to S1, OC1 to OK1
Connections:
- net +5V: now also D2.A; no longer D1.A
- net GND: now also D1.A; no longer D2.A
- net LIGHT_ON: now also IC3.PD0
- net N$3: now also D2.C; no longer D1.C
- net N$6: now also D1.C; no longer D2.C
Other:
- moved on the sheet: B1, C3, D1, D2

Commit message: PCB work
PCB TODO list work
Parts:
- renumbered JP1 to PROG, OK1 to OC1, RF1 to RF_RX

Commit message: Update receiver.sch
Parts:
- removed B1: B05S, rectifier:B05S
- added C14: 100n, resistor:C-EUC0603K
- added D3: S1G-DIO, comp_RFSwitch_v3:S1G-DIO
- added L2: 1mH, comp_RFSwitch_v3:RLB0914
- C10: value 100n -> 2.2u; device resistor:C-EUC0603K -> resistor:C-EUC1206
- C11: value 2.2u -> 10u
- C12, C8: value 10u -> 100n; device resistor:C-EUC1206 -> resistor:C-EUC0603K
- C13: value 100n -> 10u; device resistor:C-EUC0603K -> resistor:C-EUC1206
- C3: device comp_RFSwitch_v3:C-POL-EUE5-10,5 -> comp_RFSwitch_v3:C-POL-EUCAP_10X12.5_AIR
- C4: value 100n -> 4.7u; device resistor:C-EUC0603K -> comp_RFSwitch_v3:C-POL-EUE5-10,5
- C5: value 10u -> 100n; device comp_RFSwitch_v3:C_POL_PANASONIC_C_LARGER_PADS -> resistor:C-EUC0603K
- C6: value 100u -> 10u; device comp_RFSwitch_v3:C-POL_PANASONC_D_LARGER_PADS -> comp_RFSwitch_v3:C_POL_PANASONIC_C_LARGER_PADS
- C9: value 100n -> 100u; device resistor:C-EUC0603K -> comp_RFSwitch_v3:C-POL_PANASONC_D_LARGER_PADS
- D1: value US1G-DIO -> S1G-DIO; device comp_RFSwitch_v3:US1G-DIO -> comp_RFSwitch_v3:S1G-DIO
- D2: value S1G-DIO -> US1G-DIO; device comp_RFSwitch_v3:S1G-DIO -> comp_RFSwitch_v3:US1G-DIO
- IC2: value MCP1703CB -> STM8L101F2; device linear:MCP1703CB -> comp_RFSwitch_v3:STM8L101F2
- IC3: value STM8L101F2 -> MCP1703CB; device comp_RFSwitch_v3:STM8L101F2 -> linear:MCP1703CB
- R1: value 4R7 -> 10
- R5: value 1k -> 360
- R6: value 360 -> 1k
- renumbered OC1 to OK1, PROG to JP1, RF_RX to RF1
Connections:
- removed net N: B1.AC1, J1.P$2, J1.P$3
- new net N$10: C3.+, D1.C, L1.1
- net +3V3: now also C10.1, C13.1, C8.1, IC2.VDD, IC3.VO; no longer C11.1, C12.1, C9.1, IC2.VO, IC3.VDD
- net +5V: now also C11.1, C12.1, C9.+, D3.A, IC3.VI, L2.2; no longer C10.1, C6.+, C8.1, D2.A, IC2.VI, L1.2
- net BTN1: now also C14.1, IC2.PB3; no longer C13.1, IC3.PB3
- net GND: now also C14.2, C4.-, C9.-, D2.A, IC2.VSS, IC3.GND, J1.P$2, J1.P$3; no longer B1.-, C6.-, C9.2, D1.A, IC2.GND, IC3.VSS
- net LED_TX_ERR1: now also IC2.PC3; no longer IC3.PC3
- net LED_TX_ERR2: now also IC2.PC4; no longer IC3.PC4
- net LIGHT_ON: now also IC2.PB0, IC2.PD0; no longer IC3.PB0, IC3.PD0
- net LOAD: now also R5.2; no longer R6.2
- net N$1: now also C4.+, L1.2; no longer B1.+, C3.+
- net N$12: now also D1.A; no longer B1.AC2
- net N$3: now also C6.+, D3.C; no longer C5.+, D2.C
- net N$4: now also R6.2; no longer R5.2
- net N$5: now also C5.1; no longer C4.1
- net N$6: now also C5.2, C6.-, D2.C, L2.1, R6.1; no longer C4.2, C5.-, D1.C, L1.1, R5.1
- net N$7: now also R5.1; no longer R6.1
- net N$9: now also IC2.PB1; no longer IC3.PB1
- net RST: now also IC2.NRST/PA1; no longer IC3.NRST/PA1
- net SWIM: now also IC2.PA0; no longer IC3.PA0
Other:
- moved on the sheet: C10, C11, C12, C13, C3, C6, C8, D1, D2, IC1, L1, R1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

Commit message: Update receiver.sch
Parts:
- L2: device comp_RFSwitch_v3:RLB0914 -> comp_RFSwitch_v3:FERROCORE_DE0703-1000
Changed lines of the file:
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@@
 <part name="D1" library="comp_RFSwitch_v3" deviceset="S1G-DIO" device="" value="S1G-DIO"/>
 <part name="GND3" library="supply" deviceset="GND" device=""/>
-<part name="L2" library="comp_RFSwitch_v3" deviceset="RLB0914" device="" value="1mH"/>
+<part name="L2" library="comp_RFSwitch_v3" deviceset="FERROCORE_DE0703-1000" device="" value="1mH"/>
 <part name="L1" library="comp_RFSwitch_v3" deviceset="FERROCORE_DE0703-1000" device=""/>
 </parts>
