File: Remote Switch v3.1/ReceiverController/receiver.brd (EAGLE design)
At the start: 50 x 42 mm, 38 parts, among them IC1 LNK304, IC2 MCP1703CB, IC3 STM8L101F2, J1 POWER_CONN_4, T1 BT136

Commit message: PCB work - almost complete
Parts:
- C1, C11, C12, C8: device resistor:C0805K -> resistor:C1206
- C3: device resistor:E5-10,5 -> comp_RFSwitch_v3:E5-10,5
- D1: value S1G-DIO -> US1G-DIO
- D2: value US1G-DIO -> S1G-DIO
- JP1: device pinhead:1X04 -> comp_RFSwitch_v3:CON_1X4_2.54_SMD
- R1: value 10 -> 4R7; device resistor:0309/10 -> comp_RFSwitch_v3:R2512_LARGER_PADS
- R4, R6: device resistor:R0805 -> resistor:R0603
- moved R8 10.8 mm to (31.2, 5.80), flipped to the bottom, turned to 180 degrees
- moved D1 8.26 mm to (5.61, 27.8), flipped to the bottom, turned to 0 degrees
- moved D2 8.26 mm to (10.8, 21.3), flipped to the top, turned to 180 degrees
- moved C12 2.11 mm to (18.4, 10.8)
- moved R1 2.00 mm to (22.1, 40.5)
- moved C3 1.71 mm to (10.5, 37.2)
- moved C6 1.60 mm to (4.27, 17.3)
- moved C8 0.80 mm to (9.13, 15.9)
- moved B1 0.78 mm to (18.2, 35.5)
- moved C1 0.45 mm to (18.3, 3.81)
- moved C10 0.30 mm to (11.4, 15.4)
- moved C5 0.20 mm to (17.5, 19.4)
- moved C11 0.20 mm to (44.2, 7.56)
- moved IC2 0.10 mm to (14.2, 15.2)
- flipped LED1 to the bottom, turned to 0 degrees
- renumbered BTN1 to S1, OC1 to OK1
Connections:
- net +5V: now also D2.A; no longer D1.A
- net GND: now also D1.A; no longer D2.A
- net LIGHT_ON: now also IC3.9
- net N$3: now also D2.C; no longer D1.C
- net N$6: now also D1.C; no longer D2.C
Routing:
- net GND: track 120.7 -> 148.7 mm, vias 4 -> 6
- net +5V: track 8.89 -> 22.2 mm
- net BTN1: track 26.0 -> 36.5 mm, vias 0 -> 3
- net RST: track 26.8 -> 17.1 mm, vias 0 -> 1
- net N$3: track 7.80 -> 14.8 mm
- net L: track 4.60 -> 9.55 mm
- net +3V3: track 64.0 -> 67.8 mm, vias 4 -> 5
- net N$12: track 8.12 -> 4.65 mm, vias 0 -> 1
- net N$9: track 28.3 -> 31.3 mm, vias 0 -> 2
- net N$1: track 12.2 -> 10.0 mm
- net SWIM: track 19.3 -> 18.1 mm, vias 1 -> 2
- net LIGHT_ON: track 1.38 -> 2.03 mm
- net N$6: track 9.16 -> 9.73 mm

Commit message: PCB work
PCB TODO list work
Parts:
- removed RF1: RFM83/83CL, comp_RFSwitch_v3:RFM83C/83CL_CONN
- added RF_RX: RFM83/83CL, comp_RFSwitch_v3:RFM83C/83CL_CONN
- moved R8 1.57 mm to (30.4, 7.16), turned to 90 degrees
- moved R11 1.49 mm to (4.90, 9.09)
- moved C4 0.50 mm to (14.7, 26.9)
- moved C13 0.30 mm to (6.73, 9.10)
- renumbered JP1 to PROG, OK1 to OC1
Connections:
- net +3V3: now also RF_RX.4_1; no longer RF1.4_1
- net GND: now also RF_RX.2_1, RF_RX.3_1, RF_RX.6_1; no longer RF1.2_1, RF1.3_1, RF1.6_1
- net RF_DATA: now also RF_RX.5_1; no longer RF1.5_1
Routing:
- net GND: track 148.7 -> 143.2 mm, vias 6 -> 7
- net BTN1: track 36.5 -> 33.0 mm
- net +3V3: track 67.8 -> 67.0 mm
- net RST: track 17.1 -> 16.4 mm
- net N$5: track 2.30 -> 2.80 mm

Commit message: Update receiver.brd
Parts:
- removed B1: B05S, rectifier:MBS
- added C14: 100n, resistor:C0603K
- added D3: S1G-DIO, comp_RFSwitch_v3:DO214-AC
- added L2: 1mH, comp_RFSwitch_v3:RLB0914
- C10: value 100n -> 2.2u; device resistor:C0603K -> resistor:C1206
- C11: value 2.2u -> 10u
- C12, C8: value 10u -> 100n; device resistor:C1206 -> resistor:C0603K
- C13: value 100n -> 10u; device resistor:C0603K -> resistor:C1206
- C3: device comp_RFSwitch_v3:E5-10,5 -> comp_RFSwitch_v3:CAP_10X12.5_AIR
- C4: value 100n -> 4.7u; device resistor:C0603K -> comp_RFSwitch_v3:E5-10,5
- C5: value 10u -> 100n; device comp_RFSwitch_v3:PANASONIC_C_LARGER_PADS -> resistor:C0603K
- C6: value 100u -> 10u; device comp_RFSwitch_v3:PANASONIC_D_LARGER_PADS -> comp_RFSwitch_v3:PANASONIC_C_LARGER_PADS
- C9: value 100n -> 100u; device resistor:C0603K -> comp_RFSwitch_v3:PANASONIC_D_LARGER_PADS
- D1: value US1G-DIO -> S1G-DIO
- D2: value S1G-DIO -> US1G-DIO
- IC2: value MCP1703CB -> STM8L101F2; device linear:SOT23 -> comp_RFSwitch_v3:TSSOP20
- IC3: value STM8L101F2 -> MCP1703CB; device comp_RFSwitch_v3:TSSOP20 -> linear:SOT23
- R1: value 4R7 -> 10
- R5: value 1k -> 360
- R6: value 360 -> 1k
- moved C9 38.7 mm to (4.27, 16.4), turned to 90 degrees
- moved C11 36.1 mm to (9.13, 15.9)
- moved C8 33.9 mm to (42.0, 7.58)
- moved C10 33.8 mm to (44.2, 7.56)
- moved IC2 23.5 mm to (36.7, 8.24), turned to 90 degrees
- moved IC3 23.5 mm to (14.2, 15.2), turned to 0 degrees
- moved D1 22.3 mm to (24.6, 39.5), flipped to the top, turned to 270 degrees
- moved R6 17.5 mm to (16.4, 24.9)
- moved R5 17.1 mm to (33.2, 20.0)
- moved L1 14.2 mm to (15.0, 39.1), flipped to the bottom, turned to 90 degrees
- moved C6 13.9 mm to (18.1, 18.1), turned to 270 degrees
- moved C4 12.2 mm to (9.21, 37.7), flipped to the top, turned to 270 degrees
- moved C13 11.8 mm to (18.4, 10.8)
- moved C3 9.44 mm to (19.8, 35.6), turned to 270 degrees
- moved D2 9.28 mm to (5.81, 29.2), flipped to the bottom, turned to 0 degrees
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- renumbered OC1 to OK1, PROG to JP1, RF_RX to RF1
Connections:
- removed net N: B1.AC1, J1.2, J1.3
- new net N$10: C3.+, D1.C, L1.P$1
- net +3V3: now also C10.1, C13.1, C8.1, IC2.8, IC3.2; no longer C11.1, C12.1, C9.1, IC2.2, IC3.8
- net +5V: now also C11.1, C12.1, C9.+, D3.A, IC3.3, L2.2; no longer C10.1, C6.+, C8.1, D2.A, IC2.3, L1.P$2
- net BTN1: now also C14.1, IC2.13; no longer C13.1, IC3.13
- net GND: now also C14.2, C4.-, C9.-, D2.A, IC2.7, IC3.1, J1.2, J1.3; no longer B1.-, C6.-, C9.2, D1.A, IC2.1, IC3.7
- net LED_TX_ERR1: now also IC2.1; no longer IC3.1
- net LED_TX_ERR2: now also IC2.2; no longer IC3.2
- net LIGHT_ON: now also IC2.10, IC2.9; no longer IC3.10, IC3.9
- net LOAD: now also R5.2; no longer R6.2
- net N$1: now also C4.+, L1.P$2; no longer B1.+, C3.+
- net N$12: now also D1.A; no longer B1.AC2
- net N$3: now also C6.+, D3.C; no longer C5.+, D2.C
- net N$4: now also R6.2; no longer R5.2
- net N$5: now also C5.1; no longer C4.1
- net N$6: now also C5.2, C6.-, D2.C, L2.1, R6.1; no longer C4.2, C5.-, D1.C, L1.P$1, R5.1
- net N$7: now also R5.1; no longer R6.1
- net N$9: now also IC2.11; no longer IC3.11
- net RST: now also IC2.4; no longer IC3.4
- net SWIM: now also IC2.3; no longer IC3.3
Routing:
- net GND: track 143.2 -> 161.0 mm
- net N: track 16.2 -> 0.00 mm, vias 1 -> 0
- net L: track 9.55 -> 19.6 mm
- net N$10: track 0.00 -> 7.45 mm
- net N$1: track 10.0 -> 14.4 mm
- net N$12: track 4.65 -> 1.79 mm
- net BTN1: track 33.0 -> 34.9 mm
- net N$3: track 14.8 -> 16.4 mm
- net N$6: track 9.52 -> 8.33 mm, vias 16 -> 18
- net +5V: track 22.2 -> 21.2 mm
- net LOAD: vias 197 -> 229
- added copper zone on layer 1, net GND
- added copper zone on layer 16, net GND
- removed copper zone on layer 16, net L
- removed copper zone on layer 1, net N
- removed copper zone on layer 16, net N

Commit message: Update receiver.brd
Parts:
- L2: device comp_RFSwitch_v3:RLB0914 -> comp_RFSwitch_v3:DE0703
- moved L2 1.00 mm to (5.10, 26.7), turned to 270 degrees
Connections:
- net +5V: now also L2.P$2; no longer L2.2
- net N$6: now also L2.P$1; no longer L2.1
Routing:
- net +3V3: track 67.0 -> 64.3 mm, vias 5 -> 4
- net GND: track 161.0 -> 163.0 mm
- net +5V: track 21.2 -> 22.4 mm
- net N$10: track 7.45 -> 8.33 mm

Commit message: Update receiver.brd
Routing:
- net GND: track 163.0 -> 164.2 mm
Changed lines of the file:
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@@
 <contactref element="JP1" pad="3"/>
 <wire x1="1.493" y1="23.1" x2="1.493" y2="19.8" width="1.27" layer="16"/>
-<wire x1="1.493" y1="19.8" x2="1.493" y2="8.707" width="1.27" layer="16"/>
+<wire x1="1.493" y1="19.8" x2="1.493" y2="12.4" width="1.27" layer="16"/>
+<wire x1="1.493" y1="12.4" x2="1.493" y2="8.707" width="1.27" layer="16"/>
 <wire x1="39.705" y1="8.565" x2="38.365" y2="8.565" width="0.4064" layer="1"/>
 <wire x1="38.365" y1="8.565" x2="37.885" y2="8.085" width="0.4064" layer="1"/>
@@
 <wire x1="42.7" y1="6.603" x2="42.6" y2="6.703" width="1.016" layer="16"/>
 <wire x1="42.6" y1="6.703" x2="38.041" y2="6.703" width="1.016" layer="16"/>
-<wire x1="1.493" y1="8.707" x2="1.6" y2="13.5" width="0" layer="19" extent="16-16"/>
+<wire x1="1.6" y1="13.5" x2="1.493" y2="13.5" width="0.4064" layer="16"/>
+<wire x1="1.493" y1="13.5" x2="1.493" y2="12.4" width="0.4064" layer="16"/>
 </signal>
 <signal name="BTN1">
