File: Wireless_Node/wirelessnode.brd (EAGLE design)
At the start: 50 x 42 mm, 46 parts, among them IC1 LNK304, IC2 STM8L101F2, IC3 MCP1703CB, J1 POWER_CONN_4, T1 S2S4BY0F

Commit message: PCB Work, finished, final review needed
Parts:
- removed D1: S1G-DIO, comp_wirelessnode:DO214-AC
- removed R2: 4.7, resistor:R1206
- added D5: FR05JFL, semicon-smd-ipc:SOD123
- R1: value 4.7 -> CF1WS-10R; device resistor:R1206 -> comp_wirelessnode:CF1WS
- moved R1 3.00 mm to (24.5, 36.7), flipped to the top, turned to 90 degrees
- moved L1 0.10 mm to (14.6, 38.4)
Connections:
- removed net N$18: R1.2, R2.1
- net L: now also R1.2; no longer R1.1
- net N$10: now also D5.1; no longer D1.C
- net N$12: now also D5.2, R1.1; no longer D1.A, R2.2
Routing:
- net N$10: track 10.9 -> 7.26 mm
- net N$18: track 1.86 -> 0.00 mm
- net N$12: track 0.00 -> 1.69 mm
- net LOAD: track 24.5 -> 25.5 mm, vias 229 -> 222
- net N$8: track 11.2 -> 11.3 mm, vias 0 -> 1

Commit message: PCB work, almost done
Parts:
- removed D5: FR05JFL, semicon-smd-ipc:SOD123
- removed R17: 10k, resistor:R0603
- added D1: SL1G, comp_wirelessnode:SOD-123F
- added R2: 220, resistor:R0603
- D3: value S1G-DIO -> SL1G; device comp_wirelessnode:DO214-AC -> comp_wirelessnode:SOD-123F
- R10: value 3.9k -> 47
- R16: value 47 -> 10k
- R3: value 220 -> tbc
- R4: value tbc -> 360
- R6: value 360 -> 2k
- R7: value 2k -> tbc
- R8: value tbc -> 10k
- R9: value 10k -> 3.9k
- moved R9 41.5 mm to (1.96, 32.5), turned to 270 degrees
- moved R10 28.9 mm to (22.1, 11.8), turned to 180 degrees
- moved R8 22.2 mm to (36.5, 9.56), turned to 90 degrees
- moved R6 17.9 mm to (16.4, 24.9), flipped to the top, turned to 0 degrees
- moved R16 17.3 mm to (22.0, 16.3), turned to 270 degrees
- moved R4 16.9 mm to (24.6, 27.7), turned to 270 degrees
- moved R11 13.1 mm to (10.6, 5.50), turned to 270 degrees
- moved R5 11.5 mm to (33.8, 20.8), flipped to the bottom, turned to 180 degrees
- moved R3 8.82 mm to (29.6, 11.6), turned to 0 degrees
- moved R14 5.20 mm to (6.60, 5.50)
- moved R15 4.80 mm to (5.80, 10.3), turned to 180 degrees
- moved R13 4.80 mm to (12.6, 5.50)
- moved R7 3.45 mm to (19.8, 24.2), turned to 270 degrees
- moved C14 1.49 mm to (24.4, 19.8)
- moved R12 1.17 mm to (8.60, 5.50)
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- renumbered J1 to CON2
Connections:
- net +3V3: now also R16.2, R8.2; no longer R17.2, R9.2
- net +5V: now also D3.2, R9.2; no longer D3.A, R10.2
- net BTN1: now also R10.2, R16.1; no longer R11.2, R17.1
- net GND: now also R9.1; no longer R10.1
- net L: now also R4.1; no longer R5.1
- net LED_TX_ERR1: now also R2.2; no longer R3.2
- net LIGHT_ON: now also R3.1; no longer R4.1
- net LOAD: now also R5.2; no longer R6.2
- net MISO: now also R11.2; no longer R12.2
- net MOSI: now also R12.2; no longer R13.2
- net N$10: now also D1.1; no longer D5.1
- net N$11: now also R3.2; no longer R4.2
- net N$12: now also D1.2; no longer D5.2
- net N$13: now also R13.1; no longer R14.1
- net N$14: now also R12.1; no longer R13.1
- net N$15: now also R11.1; no longer R12.1
- net N$16: now also R15.1; no longer R16.1
- net N$17: now also R10.1; no longer R11.1
- net N$2: now also R2.1; no longer R3.1
- net N$3: now also D3.1, R7.2; no longer D3.C, R8.2
- net N$4: now also R6.2, R7.1; no longer R7.2, R8.1
- net N$6: now also R6.1; no longer R7.1
- net N$7: now also R5.1; no longer R6.1
- net N$8: now also R4.2; no longer R5.2
- net N$9: now also R14.1; no longer R15.1
- net NSS: now also R14.2; no longer R15.2
- net RF_RST: now also R15.2; no longer R16.2
- net RST: now also R8.1; no longer R9.1
- net SCK: now also R13.2; no longer R14.2
Routing:
- net N$9: track 18.7 -> 17.9 mm
- net N$14: track 16.6 -> 15.8 mm
- net N$13: track 11.4 -> 10.6 mm
- net L: track 19.5 -> 20.3 mm
- net N$15: track 14.4 -> 13.6 mm
- net BTN1: track 16.0 -> 16.7 mm
- net +3V3: track 45.9 -> 46.4 mm
- net GND: track 153.3 -> 153.1 mm, vias 8 -> 10

Commit message: PCB work, almost done
Parts:
- added T1OLD: S2S4BY0F, comp_wirelessnode:S2S4BY0F
- C1: value 2.2u -> 2.2u/400V
- C10: value 2.2u -> 2.2u/10V; device resistor:C1206 -> resistor:C0603K
- C11: value 10u -> 10u/25V
- C12, C14, C2, C3, C5, C7, C8: value 100n -> 100n/50V
- C13: value 10u -> 10u/6.3V; device resistor:C1206 -> resistor:C0603K
- C4: value 4.7u -> 4.7u/400V
- C6: value 4.7u -> 4.7u/50V
- C9: value 100u -> 100u/35V
- CON1: device comp_wirelessnode:CON_1X4_1.27_SMD -> CarReceiver:TERMINAL_BLOCK_4
- CON2: value POWER_CONN_4 -> ZL321-4P; device CarReceiver:TERMINAL_BLOCK_4 -> comp_wirelessnode:CON_1X4_1.27_SMD
- D1, D3: value SL1G -> 1A/400V
- D2: value US1G-DIO -> 1A/400V
- IC3: value MCP1703CB -> MCP1703
- L1: value FERROCORE_DE0703-1000 -> 1mH
- LED1: value (none) -> RED/GREEN
- R1: value CF1WS-10R -> 10
- R7: value tbc -> 8.6K
- R9: value 3.9k -> 3.3k
- S1: value B3F-1050 -> SPST-NO
- T1: value S2S4BY0F -> MOC3042S; device comp_wirelessnode:S2S4BY0F -> optocoupler:DIL6-SMD
- T2: value (none) -> BTA16
- moved CON2 34.0 mm to (40.4, 5.20), turned to 0 degrees
- moved CON1 30.5 mm to (36.6, 39.0), turned to 270 degrees
- moved R14 16.7 mm to (22.1, 11.8), turned to 180 degrees
- moved R10 13.1 mm to (10.6, 5.50), turned to 270 degrees
- moved LED1 6.87 mm to (32.4, 3.30), turned to 180 degrees
- moved R13 6.00 mm to (6.60, 5.50)
- moved R12 4.00 mm to (12.6, 5.50)
- moved T1 3.19 mm to (34.1, 14.0), turned to 0 degrees
- moved R5 2.79 mm to (36.6, 21.1), turned to 90 degrees
- moved C14 2.40 mm to (24.4, 17.4)
- moved S1 2.30 mm to (24.4, 14.6)
- moved R11 1.97 mm to (8.60, 5.50)
- moved C8 0.76 mm to (31.3, 8.38)
- moved C10 0.76 mm to (33.5, 8.36)
- moved C13 0.20 mm to (17.1, 12.1)
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Connections:
- net +5V renamed +9.2V
- net +3V3: now also CON2.1; no longer CON1.1
- net BTN1: now also R14.2, S1.3, S1.4; no longer R10.2, S1.P$3, S1.P$4
- net GND: now also CON1.2, S1.1, S1.2; no longer CON2.2, S1.P$1, S1.P$2
- net L: now also CON1.4; no longer CON2.4
- net LOAD: now also CON1.1; no longer CON2.1
- net MISO: now also R10.2; no longer R11.2
- net MOSI: now also R11.2; no longer R12.2
- net N$13: now also R12.1; no longer R13.1
- net N$14: now also R11.1; no longer R12.1
- net N$15: now also R10.1; no longer R11.1
- net N$17: now also R14.1; no longer R10.1
- net N$7: now also T1.6; no longer T1.4
- net N$8: now also T1.4; no longer T1.3
- net N$9: now also R13.1; no longer R14.1
- net NSS: now also R13.2; no longer R14.2
- net RST: now also CON2.4; no longer CON1.4
- net SCK: now also R12.2; no longer R13.2
- net SWIM: now also CON2.2; no longer CON1.2
Routing:
- net N$2: track 9.72 -> 1.77 mm
- net LED_TX_ERR2: track 11.3 -> 5.82 mm
- net N$11: track 3.27 -> 7.60 mm
- net GND: track 153.1 -> 149.2 mm, vias 10 -> 9
- net +3V3: track 46.4 -> 50.2 mm
- net BTN1: track 16.7 -> 15.0 mm
- net RST: track 24.1 -> 25.3 mm
- net SWIM: track 13.5 -> 12.7 mm
- net N$8: track 11.3 -> 11.9 mm, vias 1 -> 0
- net LOAD: track 25.5 -> 25.1 mm, vias 222 -> 221

Commit message: PCB work
Parts:
- removed T1OLD: S2S4BY0F, comp_wirelessnode:S2S4BY0F
- LED1: device led:LED3MM -> led:LED5MM
- R3: value tbc -> 220
- T1: value MOC3042S -> MOC3063XSM
- moved R14 1.40 mm to (20.7, 11.8)
- moved LED1 1.36 mm to (33.2, 4.40), turned to 0 degrees
- moved C8 0.98 mm to (31.7, 9.28)
- moved C10 0.91 mm to (33.6, 9.26)
- moved R3 0.64 mm to (29.1, 12.0)
- moved R8 0.30 mm to (36.5, 9.26)
Routing:
- net N$2: track 1.77 -> 5.56 mm
- net LED_TX_ERR2: track 5.82 -> 3.62 mm
- net RST: track 25.3 -> 23.7 mm
- net BTN1: track 15.0 -> 16.3 mm
- net N$17: track 5.68 -> 6.40 mm
- net N$11: track 7.60 -> 8.27 mm
- net LOAD: vias 221 -> 214

Commit message: PCB work, finished
Parts:
- C13: value 10u/6.3V -> 10u/10V
- T1: value MOC3063XSM -> VO3063-X007T
- T2: device comp_wirelessnode:TO220 -> comp_wirelessnode:TO220_SMD
Routing:
- net LOAD: track 25.1 -> 23.7 mm, vias 214 -> 218
- net N$8: track 11.9 -> 12.4 mm, vias 0 -> 1
