File: Wireless_Node/wirelessnode.sch (EAGLE design)
At the start: 46 parts, among them IC1 LNK304, IC2 STM8L101F2, IC3 MCP1703CB, J1 POWER_CONN_4, T1 S2S4BY0F

Commit message: PCB Work, finished, final review needed
Parts:
- removed D1: S1G-DIO, comp_wirelessnode:S1G-DIO
- removed R2: 4.7, resistor:R-EU_R1206
- added D5: FR05JFL, semicon-smd-ipc:D-SOD123
- R1: value 4.7 -> CF1WS-10R; device resistor:R-EU_R1206 -> comp_wirelessnode:R_CF1WS
Connections:
- removed net N$18: R1.2, R2.1
- net L: now also R1.2; no longer R1.1
- net N$10: now also D5.C; no longer D1.C
- net N$12: now also D5.A, R1.1; no longer D1.A, R2.2
Other:
- moved on the sheet: R1
Changed lines of the file:
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@@
 <grid distance="0.1" unitdist="inch" unit="inch" style="lines" multiple="1" display="no" altdistance="0.01" altunitdist="inch" altunit="inch"/>
 <layers>
-<layer number="1" name="Top" color="4" fill="1" visible="yes" active="no"/>
-<layer number="16" name="Bottom" color="1" fill="1" visible="yes" active="no"/>
-<layer number="17" name="Pads" color="2" fill="1" visible="yes" active="no"/>
-<layer number="18" name="Vias" color="2" fill="1" visible="yes" active="no"/>
-<layer number="19" name="Unrouted" color="6" fill="1" visible="yes" active="no"/>
-<layer number="20" name="Dimension" color="15" fill="1" visible="yes" active="no"/>
-<layer number="21" name="tPlace" color="7" fill="1" visible="yes" active="no"/>
-<layer number="22" name="bPlace" color="7" fill="1" visible="yes" active="no"/>
-<layer number="23" name="tOrigins" color="15" fill="1" visible="yes" active="no"/>
-<layer number="24" name="bOrigins" color="15" fill="1" visible="yes" active="no"/>
-<layer number="25" name="tNames" color="7" fill="1" visible="yes" active="no"/>
-<layer number="26" name="bNames" color="7" fill="1" visible="yes" active="no"/>
-<layer number="27" name="tValues" color="7" fill="1" visible="yes" active="no"/>
-<layer number="28" name="bValues" color="7" fill="1" visible="yes" active="no"/>
+<layer number="1" name="Top" color="4" fill="1" visible="no" active="no"/>
+<layer number="16" name="Bottom" color="1" fill="1" visible="no" active="no"/>
+<layer number="17" name="Pads" color="2" fill="1" visible="no" active="no"/>
+<layer number="18" name="Vias" color="2" fill="1" visible="no" active="no"/>
+<layer number="19" name="Unrouted" color="6" fill="1" visible="no" active="no"/>
+<layer number="20" name="Dimension" color="15" fill="1" visible="no" active="no"/>
+<layer number="21" name="tPlace" color="7" fill="1" visible="no" active="no"/>
+<layer number="22" name="bPlace" color="7" fill="1" visible="no" active="no"/>
+<layer number="23" name="tOrigins" color="15" fill="1" visible="no" active="no"/>
+<layer number="24" name="bOrigins" color="15" fill="1" visible="no" active="no"/>
+<layer number="25" name="tNames" color="7" fill="1" visible="no" active="no"/>
+<layer number="26" name="bNames" color="7" fill="1" visible="no" active="no"/>
+<layer number="27" name="tValues" color="7" fill="1" visible="no" active="no"/>
+<layer number="28" name="bValues" color="7" fill="1" visible="no" active="no"/>
 <layer number="29" name="tStop" color="7" fill="3" visible="no" active="no"/>
 <layer number="30" name="bStop" color="7" fill="6" visible="no" active="no"/>
@@
 <layer number="35" name="tGlue" color="7" fill="4" visible="no" active="no"/>
 <layer number="36" name="bGlue" color="7" fill="5" visible="no" active="no"/>
-<layer number="37" name="tTest" color="7" fill="1" visible="yes" active="no"/>
-<layer number="38" name="bTest" color="7" fill="1" visible="yes" active="no"/>
+<layer number="37" name="tTest" color="7" fill="1" visible="no" active="no"/>
+<layer number="38" name="bTest" color="7" fill="1" visible="no" active="no"/>
 <layer number="39" name="tKeepout" color="4" fill="11" visible="no" active="no"/>
 <layer number="40" name="bKeepout" color="1" fill="11" visible="no" active="no"/>
@@
 <layer number="44" name="Drills" color="7" fill="1" visible="no" active="no"/>
 <layer number="45" name="Holes" color="7" fill="1" visible="no" active="no"/>
-<layer number="46" name="Milling" color="3" fill="1" visible="yes" active="no"/>
-<layer number="47" name="Measures" color="7" fill="1" visible="yes" active="no"/>
-<layer number="48" name="Document" color="7" fill="1" visible="yes" active="no"/>
-<layer number="49" name="Reference" color="7" fill="1" visible="yes" active="no"/>
-<layer number="50" name="dxf" color="7" fill="1" visible="yes" active="no"/>
-<layer number="51" name="tDocu" color="7" fill="1" visible="yes" active="no"/>
-<layer number="52" name="bDocu" color="7" fill="1" visible="yes" active="no"/>
-<layer number="53" name="tGND_GNDA" color="7" fill="9" visible="yes" active="no"/>
-<layer number="54" name="bGND_GNDA" color="1" fill="9" visible="yes" active="no"/>
-<layer number="56" name="wert" color="7" fill="1" visible="yes" active="no"/>
+<layer number="46" name="Milling" color="3" fill="1" visible="no" active="no"/>
+<layer number="47" name="Measures" color="7" fill="1" visible="no" active="no"/>
+<layer number="48" name="Document" color="7" fill="1" visible="no" active="no"/>
+<layer number="49" name="Reference" color="7" fill="1" visible="no" active="no"/>
+<layer number="50" name="dxf" color="7" fill="1" visible="no" active="no"/>
+<layer number="51" name="tDocu" color="7" fill="1" visible="no" active="no"/>
+<layer number="52" name="bDocu" color="7" fill="1" visible="no" active="no"/>
+<layer number="53" name="tGND_GNDA" color="7" fill="9" visible="no" active="no"/>
+<layer number="54" name="bGND_GNDA" color="1" fill="9" visible="no" active="no"/>
+<layer number="56" name="wert" color="7" fill="1" visible="no" active="no"/>
 <layer number="90" name="Modules" color="5" fill="1" visible="no" active="no"/>
 <layer number="91" name="Nets" color="2" fill="1" visible="yes" active="yes"/>
@@
 <part name="C1" library="comp_wirelessnode" deviceset="C-POL-EU" device="CAP_8X11.5_AIR" value="2.2u"/>
 <part name="GND2" library="supply" deviceset="GND" device=""/>
-<part name="D1" library="comp_wirelessnode" deviceset="S1G-DIO" device="" value="S1G-DIO"/>
 <part name="GND1" library="supply" deviceset="GND" device=""/>
 <part name="L2" library="comp_wirelessnode" deviceset="FERROCORE_DE0703-1000" device="" value="1mH"/>
@@
 <part name="T1" library="comp_wirelessnode" deviceset="S2S4BY0F" device="" value="S2S4BY0F"/>
 <part name="R11" library="resistor" deviceset="R-EU_" device="R0603" value="47"/>
-<part name="R2" library="resistor" deviceset="R-EU_" device="R1206" value="4.7"/>
-<part name="R1" library="resistor" deviceset="R-EU_" device="R1206" value="4.7"/>
+<part name="R1" library="comp_wirelessnode" deviceset="R_" device="CF1WS" value="CF1WS-10R"/>
+<part name="D5" library="semicon-smd-ipc" deviceset="D-" device="SOD123" value="FR05JFL"/>
 </parts>
 <sheets>
@@
 <instance part="C1" gate="G$1" x="58.42" y="33.02"/>
 <instance part="GND2" gate="1" x="58.42" y="25.4"/>
-<instance part="D1" gate="G$1" x="50.8" y="35.56"/>
 <instance part="GND1" gate="1" x="35.56" y="25.4"/>
 <instance part="L2" gate="G$1" x="139.7" y="50.8"/>
@@
 <instance part="T1" gate="G$1" x="76.2" y="129.54"/>
 <instance part="R11" gate="G$1" x="218.44" y="111.76"/>
-<instance part="R2" gate="G$1" x="43.18" y="35.56"/>
-<instance part="R1" gate="G$1" x="33.02" y="35.56"/>
+<instance part="R1" gate="G$1" x="40.64" y="35.56" rot="R180"/>
+<instance part="D5" gate="G$1" x="53.34" y="35.56"/>
 </instances>
 <busses>
@@
 </segment>
 <segment>
-<wire x1="27.94" y1="35.56" x2="20.32" y2="35.56" width="0.1524" layer="91"/>
-<label x="20.32" y="35.56" size="1.778" layer="95"/>
-<pinref part="R1" gate="G$1" pin="1"/>
-</segment>
-<segment>
 <pinref part="J1" gate="G$1" pin="P$4"/>
 <wire x1="22.86" y1="121.92" x2="27.94" y2="121.92" width="0.1524" layer="91"/>
 <label x="25.4" y="121.92" size="1.778" layer="95"/>
+</segment>
+<segment>
+<pinref part="R1" gate="G$1" pin="2"/>
+<wire x1="35.56" y1="35.56" x2="20.32" y2="35.56" width="0.1524" layer="91"/>
+<label x="20.32" y="35.56" size="1.778" layer="95"/>
 </segment>
 </net>
@@
 <net name="N$10" class="0">
 <segment>
-<pinref part="D1" gate="G$1" pin="C"/>
 <pinref part="C1" gate="G$1" pin="+"/>
-<wire x1="53.34" y1="35.56" x2="58.42" y2="35.56" width="0.1524" layer="91"/>
 <pinref part="L1" gate="G$1" pin="1"/>
 <wire x1="60.96" y1="35.56" x2="58.42" y2="35.56" width="0.1524" layer="91"/>
+<pinref part="D5" gate="G$1" pin="C"/>
+<wire x1="55.88" y1="35.56" x2="58.42" y2="35.56" width="0.1524" layer="91"/>
 <junction x="58.42" y="35.56"/>
 </segment>
@@
 <net name="N$12" class="0">
 <segment>
-<pinref part="D1" gate="G$1" pin="A"/>
-<pinref part="R2" gate="G$1" pin="2"/>
-</segment>
-</net>
-<net name="N$18" class="0">
-<segment>
-<pinref part="R2" gate="G$1" pin="1"/>
-<pinref part="R1" gate="G$1" pin="2"/>
-</segment>
-</net>
+<pinref part="D5" gate="G$1" pin="A"/>
+<pinref part="R1" gate="G$1" pin="1"/>
+<wire x1="50.8" y1="35.56" x2="45.72" y2="35.56" width="0.1524" layer="91"/>
+</segment>
+</net>

Commit message: PCB work, almost done
Parts:
- removed D5: FR05JFL, semicon-smd-ipc:D-SOD123
- removed R17: 10k, resistor:R-EU_R0603
- added D1: SL1G, comp_wirelessnode:SL1G
- added R2: 220, resistor:R-EU_R0603
- D3: value S1G-DIO -> SL1G; device comp_wirelessnode:S1G-DIO -> comp_wirelessnode:SL1G
- R10: value 3.9k -> 47
- R16: value 47 -> 10k
- R3: value 220 -> tbc
- R4: value tbc -> 360
- R6: value 360 -> 2k
- R7: value 2k -> tbc
- R8: value tbc -> 10k
- R9: value 10k -> 3.9k
- renumbered J1 to CON2
Connections:
- net +3V3: now also R16.2, R8.2; no longer R17.2, R9.2
- net +5V: now also R9.2; no longer R10.2
- net BTN1: now also R10.2, R16.1; no longer R11.2, R17.1
- net GND: now also R9.1; no longer R10.1
- net L: now also R4.1; no longer R5.1
- net LED_TX_ERR1: now also R2.2; no longer R3.2
- net LIGHT_ON: now also R3.1; no longer R4.1
- net LOAD: now also R5.2; no longer R6.2
- net MISO: now also R11.2; no longer R12.2
- net MOSI: now also R12.2; no longer R13.2
- net N$10: now also D1.C; no longer D5.C
- net N$11: now also R3.2; no longer R4.2
- net N$12: now also D1.A; no longer D5.A
- net N$13: now also R13.1; no longer R14.1
- net N$14: now also R12.1; no longer R13.1
- net N$15: now also R11.1; no longer R12.1
- net N$16: now also R15.1; no longer R16.1
- net N$17: now also R10.1; no longer R11.1
- net N$2: now also R2.1; no longer R3.1
- net N$3: now also R7.2; no longer R8.2
- net N$4: now also R6.2, R7.1; no longer R7.2, R8.1
- net N$6: now also R6.1; no longer R7.1
- net N$7: now also R5.1; no longer R6.1
- net N$8: now also R4.2; no longer R5.2
- net N$9: now also R14.1; no longer R15.1
- net NSS: now also R14.2; no longer R15.2
- net RF_RST: now also R15.2; no longer R16.2
- net RST: now also R8.1; no longer R9.1
- net SCK: now also R13.2; no longer R14.2
Other:
- moved on the sheet: R10, R11, R12, R13, R14, R15, R16, R3, R4, R5, R6, R7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

Commit message: PCB work, almost done
Parts:
- added T1OLD: S2S4BY0F, comp_wirelessnode:S2S4BY0F
- C1: value 2.2u -> 2.2u/400V; TME_ORDER_NUMBER (none) -> RD2G225M0811MBB
- C10: value 2.2u -> 2.2u/10V; device resistor:C-EUC1206 -> resistor:C-EUC0603K; TME_ORDER_NUMBER (none) -> CL10A225KP8NNNC
- C11: value 10u -> 10u/25V; TME_ORDER_NUMBER (none) -> 08053D106KAT2A
- C12, C14, C2, C3, C5, C7, C8: value 100n -> 100n/50V; TME_ORDER_NUMBER (none) -> C0603C104K5RAC
- C13: value 10u -> 10u/6.3V; device resistor:C-EUC1206 -> resistor:C-EUC0603K; TME_ORDER_NUMBER (none) -> CL10A106KQ8NNNC
- C4: value 4.7u -> 4.7u/400V; TME_ORDER_NUMBER (none) -> RD2G475M1012MBB
- C6: value 4.7u -> 4.7u/50V; TME_ORDER_NUMBER (none) -> RC1H475M05005VR
- C9: value 100u -> 100u/35V; TME_ORDER_NUMBER (none) -> UCD1V101MCL6GS
- CON1: value (none) -> POWER_CONN_4; device comp_wirelessnode:CON_1X4PIN_1.27MM_SMD -> CarReceiver:POWER_CONN_4; TME_ORDER_NUMBER (none) -> EBBA-02-C-SS-BU
- CON2: value POWER_CONN_4 -> ZL321-4P; device CarReceiver:POWER_CONN_4 -> comp_wirelessnode:CON_1X4PIN_1.27MM_SMD; TME_ORDER_NUMBER (none) -> ZL321-4P (DS1065-01-1X4S8BV)
- D1, D3: value SL1G -> 1A/400V; TME_ORDER_NUMBER (none) -> SL1G-DIO
- D2: value US1G-DIO -> 1A/400V; TME_ORDER_NUMBER (none) -> US1G-DIO
- IC1: TME_ORDER_NUMBER (none) -> LNK304DN
- IC2: TME_ORDER_NUMBER (none) -> STM8L101F2P6
- IC3: value MCP1703CB -> MCP1703; TME_ORDER_NUMBER (none) -> MCP1703T3302ECB
- L1: value FERROCORE_DE0703-1000 -> 1mH; TME_ORDER_NUMBER (none) -> DE0703-1000
- L2: TME_ORDER_NUMBER (none) -> DE0703-1000
- LED1: value (none) -> RED/GREEN; TME_ORDER_NUMBER (none) -> L-937EGW
- R1: value CF1WS-10R -> 10; TME_ORDER_NUMBER (none) -> CF1WS-10R
- R7: value tbc -> 8.6K
- R9: value 3.9k -> 3.3k
- RF1: TME_ORDER_NUMBER (none) -> RFM69HW-868S2
- S1: value B3F-1050 -> SPST-NO; TME_ORDER_NUMBER (none) -> DTSM-63N-V-B
- T1: value S2S4BY0F -> MOC3042S; device comp_wirelessnode:S2S4BY0F -> optocoupler:MOC3042S
- T2: value (none) -> BTA16; TME_ORDER_NUMBER (none) -> BTA16-600BRG
Connections:
- net +5V renamed +9.2V
- net +3V3: now also CON2.1; no longer CON1.1
- net BTN1: now also R14.2; no longer R10.2
- net GND: now also CON1.P$2, CON1.P$3, CON2.3; no longer CON1.3, CON2.P$2, CON2.P$3
- net L: now also CON1.P$4; no longer CON2.P$4
- net LOAD: now also CON1.P$1; no longer CON2.P$1
- net MISO: now also R10.2; no longer R11.2
- net MOSI: now also R11.2; no longer R12.2
- net N$13: now also R12.1; no longer R13.1
- net N$14: now also R11.1; no longer R12.1
- net N$15: now also R10.1; no longer R11.1
- net N$17: now also R14.1; no longer R10.1
- net N$9: now also R13.1; no longer R14.1
- net NSS: now also R13.2; no longer R14.2
- net RST: now also CON2.4; no longer CON1.4
- net SCK: now also R12.2; no longer R13.2
- net SWIM: now also CON2.2; no longer CON1.2
Other:
- note added: "LED current = 21mA"
- moved on the sheet: C11, C12, C13, C8, CON1, CON2, D1, IC3, R1, R10, R11, R12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

Commit message: PCB work
Parts:
- removed T1OLD: S2S4BY0F, comp_wirelessnode:S2S4BY0F
- LED1: device led:LED3MM -> led:LED5MM; TME_ORDER_NUMBER L-937EGW -> L-57EGW
- R3: value tbc -> 220
- T1: value MOC3042S -> MOC3063XSM; TME_ORDER_NUMBER (none) -> MOC3063XSM
Other:
- note added: "LED current = 10mA"
- note removed: "LED current = 21mA"
Changed lines of the file:
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@@
 <part name="+3V34" library="supply1" deviceset="+3V3" device=""/>
 <part name="GND17" library="supply" deviceset="GND" device=""/>
-<part name="LED1" library="led" deviceset="LED" device="3MM" value="RED/GREEN">
-<attribute name="TME_ORDER_NUMBER" value="L-937EGW"/>
+<part name="LED1" library="led" deviceset="LED" device="5MM" value="RED/GREEN">
+<attribute name="TME_ORDER_NUMBER" value="L-57EGW"/>
 </part>
 <part name="C10" library="resistor" deviceset="C-EU" device="C0603K" value="2.2u/10V">
@@
 <part name="R5" library="resistor" deviceset="R-EU_" device="R0603" value="360"/>
 <part name="R4" library="resistor" deviceset="R-EU_" device="R0603" value="360"/>
-<part name="R3" library="resistor" deviceset="R-EU_" device="R0603" value="tbc"/>
+<part name="R3" library="resistor" deviceset="R-EU_" device="R0603" value="220"/>
 <part name="GND3" library="supply" deviceset="GND" device=""/>
 <part name="IC3" library="linear" deviceset="MCP1703" device="CB" value="MCP1703">
@@
 <part name="R13" library="resistor" deviceset="R-EU_" device="R0603" value="47"/>
 <part name="R15" library="resistor" deviceset="R-EU_" device="R0603" value="47"/>
-<part name="T1OLD" library="comp_wirelessnode" deviceset="S2S4BY0F" device="" value="S2S4BY0F">
-<attribute name="TME_ORDER_NUMBER" value="S2S4BY0F"/>
-</part>
 <part name="R14" library="resistor" deviceset="R-EU_" device="R0603" value="47"/>
 <part name="R1" library="comp_wirelessnode" deviceset="R_" device="CF1WS" value="10">
@@
 <attribute name="TME_ORDER_NUMBER" value="SL1G-DIO"/>
 </part>
-<part name="T1" library="optocoupler" deviceset="MOC30*" device="S" technology="42"/>
+<part name="T1" library="optocoupler" deviceset="MOC30*" device="S" technology="42" value="MOC3063XSM">
+<attribute name="TME_ORDER_NUMBER" value="MOC3063XSM"/>
+</part>
 </parts>
 <sheets>
 <sheet>
 <plain>
-<text x="48.26" y="127" size="1.778" layer="97">LED current = 21mA</text>
+<text x="48.26" y="127" size="1.778" layer="97">LED current = 10mA</text>
 </plain>
 <instances>
@@
 <instance part="R13" gate="G$1" x="220.98" y="114.3"/>
 <instance part="R15" gate="G$1" x="220.98" y="106.68"/>
-<instance part="T1OLD" gate="G$1" x="119.38" y="149.86">
-<attribute name="TME_ORDER_NUMBER" x="119.38" y="149.86" size="1.778" layer="96" display="off"/>
-</instance>
 <instance part="R14" gate="G$1" x="220.98" y="111.76"/>
 <instance part="R1" gate="G$1" x="38.1" y="35.56" smashed="yes" rot="R180">
@@
 <attribute name="TME_ORDER_NUMBER" x="48.26" y="35.56" size="1.778" layer="96" display="off"/>
 </instance>
-<instance part="T1" gate="-1" x="81.28" y="129.54"/>
+<instance part="T1" gate="-1" x="81.28" y="129.54">
+<attribute name="TME_ORDER_NUMBER" x="81.28" y="129.54" size="1.778" layer="96" display="off"/>
+</instance>
 </instances>
 <busses>
@@
 <segment>
 <pinref part="LED1" gate="G$1" pin="C"/>
-<wire x1="48.26" y1="162.56" x2="48.26" y2="157.48" width="0.1524" layer="91"/>
-<wire x1="48.26" y1="157.48" x2="81.28" y2="157.48" width="0.1524" layer="91"/>
+<wire x1="48.26" y1="162.56" x2="48.26" y2="154.94" width="0.1524" layer="91"/>
+<wire x1="48.26" y1="154.94" x2="81.28" y2="154.94" width="0.1524" layer="91"/>
 <label x="66.04" y="157.48" size="1.778" layer="95"/>
 </segment>

Commit message: PCB work, finished
Parts:
- C13: value 10u/6.3V -> 10u/10V; TME_ORDER_NUMBER CL10A106KQ8NNNC -> 0603ZD106MAT2A
- R6: TME_ORDER_NUMBER (none) -> RC0603FR-072K
- R7: TME_ORDER_NUMBER (none) -> CRCW06038K66FKTABC
- R9: TME_ORDER_NUMBER (none) -> RC0603FR-073K3
- T1: value MOC3063XSM -> VO3063-X007T; TME_ORDER_NUMBER MOC3063XSM -> VO3063-X007T
- T2: device comp_wirelessnode:BT136 -> comp_wirelessnode:BT136SMD
Changed lines of the file:
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@@
 <?xml version="1.0" encoding="utf-8"?>
 <!DOCTYPE eagle SYSTEM "eagle.dtd">
-<eagle version="7.3.0">
+<eagle version="7.5.0">
 <drawing>
 <settings>
@@
 </part>
 <part name="FRAME1" library="frames" deviceset="A4L-LOC" device="" value="EmitterSwitch"/>
-<part name="R9" library="resistor" deviceset="R-EU_" device="R0603" value="3.3k"/>
+<part name="R9" library="resistor" deviceset="R-EU_" device="R0603" value="3.3k">
+<attribute name="TME_ORDER_NUMBER" value="RC0603FR-073K3"/>
+</part>
 <part name="C4" library="comp_RFSwitch_v3" deviceset="C-POL-EU" device="E5-10,5" value="4.7u/400V">
 <attribute name="TME_ORDER_NUMBER" value="RD2G475M1012MBB"/>
@@
 <attribute name="TME_ORDER_NUMBER" value="RC1H475M05005VR"/>
 </part>
-<part name="R7" library="resistor" deviceset="R-EU_" device="R0603" value="8.6K"/>
-<part name="R6" library="resistor" deviceset="R-EU_" device="R0603" value="2k"/>
-<part name="T2" library="comp_wirelessnode" deviceset="BT136" device="" value="BTA16">
+<part name="R7" library="resistor" deviceset="R-EU_" device="R0603" value="8.6K">
+<attribute name="TME_ORDER_NUMBER" value="CRCW06038K66FKTABC "/>
+</part>
+<part name="R6" library="resistor" deviceset="R-EU_" device="R0603" value="2k">
+<attribute name="TME_ORDER_NUMBER" value="RC0603FR-072K"/>
+</part>
+<part name="T2" library="comp_wirelessnode" deviceset="BT136" device="SMD" value="BTA16">
 <attribute name="TME_ORDER_NUMBER" value="BTA16-600BRG"/>
 </part>
@@
 <attribute name="TME_ORDER_NUMBER" value="MCP1703T3302ECB"/>
 </part>
-<part name="C13" library="resistor" deviceset="C-EU" device="C0603K" value="10u/6.3V">
-<attribute name="TME_ORDER_NUMBER" value="CL10A106KQ8NNNC"/>
+<part name="C13" library="resistor" deviceset="C-EU" device="C0603K" value="10u/10V">
+<attribute name="TME_ORDER_NUMBER" value="0603ZD106MAT2A"/>
 </part>
 <part name="GND18" library="supply" deviceset="GND" device=""/>
@@
 <attribute name="TME_ORDER_NUMBER" value="SL1G-DIO"/>
 </part>
-<part name="T1" library="optocoupler" deviceset="MOC30*" device="S" technology="42" value="MOC3063XSM">
-<attribute name="TME_ORDER_NUMBER" value="MOC3063XSM"/>
+<part name="T1" library="optocoupler" deviceset="MOC30*" device="S" technology="42" value="VO3063-X007T">
+<attribute name="TME_ORDER_NUMBER" value="VO3063-X007T"/>
 </part>
 </parts>
@@
 </instance>
 <instance part="FRAME1" gate="G$1" x="0" y="0"/>
-<instance part="R9" gate="G$1" x="170.18" y="45.72" rot="R90"/>
+<instance part="R9" gate="G$1" x="170.18" y="45.72" rot="R90">
+<attribute name="TME_ORDER_NUMBER" x="170.18" y="45.72" size="1.778" layer="96" rot="R90" display="off"/>
+</instance>
 <instance part="C4" gate="G$1" x="78.74" y="33.02">
 <attribute name="TME_ORDER_NUMBER" x="78.74" y="33.02" size="1.778" layer="96" display="off"/>
@@
 <attribute name="TME_ORDER_NUMBER" x="129.54" y="63.5" size="1.778" layer="96" display="off"/>
 </instance>
-<instance part="R7" gate="G$1" x="121.92" y="66.04"/>
-<instance part="R6" gate="G$1" x="114.3" y="60.96" rot="R90"/>
+<instance part="R7" gate="G$1" x="121.92" y="66.04">
+<attribute name="TME_ORDER_NUMBER" x="121.92" y="66.04" size="1.778" layer="96" display="off"/>
+</instance>
+<instance part="R6" gate="G$1" x="114.3" y="60.96" rot="R90">
+<attribute name="TME_ORDER_NUMBER" x="114.3" y="60.96" size="1.778" layer="96" rot="R90" display="off"/>
+</instance>
 <instance part="T2" gate="G$1" x="104.14" y="127">
 <attribute name="TME_ORDER_NUMBER" x="104.14" y="127" size="1.778" layer="96" display="off"/>
