File: Wireless_Node/Relay/wirelessnode_relay.sch (EAGLE design)
At the start: 48 parts, among them CON1 ZL321-4P, IC1 LNK304, IC2 DS18B20, IC3 STM8L101F2, IC4 MCP1703, J1 POWER_CONN_4, T1 BC817

Commit message: Ready for production
Parts:
- removed D5: 1A/400V, comp_wirelessnode:SL1G
- removed J1: POWER_CONN_4, CarReceiver:POWER_CONN_4
- added B1: B05S, rectifier:B05S
- added C15: (no value), resistor:C-EUC1812
- added CON2: ZL321-4P, comp_wirelessnode:CON_1X4PIN_1.27MM_SMD
- added R17: (no value), resistor:R-EU_R2010
- C4: value 4.7u/400V -> 2.2u/400V; device comp_RFSwitch_v3:C-POL-EUE5-10,5 -> comp_wirelessnode:C-POL-EUE3.5-8; TME_ORDER_NUMBER RD2G475M1012MBB -> RD2G225M0811MBB
- CON1: value ZL321-4P -> POWER_CONN_4; device comp_wirelessnode:CON_1X4PIN_1.27MM_SMD -> CarReceiver:POWER_CONN_4; TME_ORDER_NUMBER ZL321-4P (DS1065-01-1X4S8BV) -> EBBA-02-C-SS-BU
- D1: value 1A/400V -> BAS16HT1G; device comp_wirelessnode:SL1G -> diode:DIODE-SOD323-W; TME_ORDER_NUMBER SL1G-DIO -> BAS16HT1G
- D3: value BAS16HT1G -> 1A/400V; device diode:DIODE-SOD323-W -> comp_wirelessnode:US1G-DIO; TME_ORDER_NUMBER BAS16HT1G -> US1G-DIO
- D4: device comp_wirelessnode:US1G-DIO -> comp_wirelessnode:SL1G; TME_ORDER_NUMBER US1G-DIO -> SL1G-DIO
Connections:
- removed net LOAD: J1.P$1, K1G$2.S
- new net N: B1.AC2, CON1.P$3
- new net N$12: C15.2, R17.2
- new net SW1: C15.1, CON1.P$1, K1G$2.S
- new net SW2: CON1.P$2, K1G$2.P, R17.1
- net +12V: now also D1.C, D4.A; no longer D2.C, D5.A
- net +3V3: now also CON2.1; no longer CON1.1
- net GND: now also B1.-, CON2.3, D2.A; no longer CON1.3, D4.A, J1.P$2, J1.P$3
- net L: now also CON1.P$4; no longer J1.P$4, K1G$2.P
- net N$10: now also B1.+; no longer D1.C
- net N$3: now also D4.C; no longer D5.C
- net N$6: now also D3.C; no longer D4.C
- net N$7: now also B1.AC1; no longer D1.A
- net N$8: now also D1.A, D2.C; no longer D2.A, D3.C
- net RST: now also CON2.4; no longer CON1.4
- net SWIM: now also CON2.2; no longer CON1.2
Other:
- moved on the sheet: CON1, D1, D2, D3, D4, K1, R1
