File: Wireless_Node/Triac/wirelessnode_triac.brd (EAGLE design)
At the start: 50 x 42 mm, 48 parts, among them CON2 ZL321-4P, IC1 LNK304, IC2 STM8L101F2, IC3 MCP1703, IC4 DS18B20, T1 VO3063-X007T, T2 BTA16

Commit message: Ready for production
Parts:
- removed D3: 1A/400V, comp_wirelessnode:SOD-123F
- removed T2: BTA16, comp_wirelessnode:TO220_SMD
- added B1: B05S, rectifier:MBS
- added OK1: VO3063-X007T, optocoupler:DIL6-SMD
- C1: device comp_wirelessnode:CAP_8X11.5_AIR -> comp_wirelessnode:E3.5-8
- C4: value 4.7u/400V -> 2.2u/400V; device comp_RFSwitch_v3:E5-10,5 -> comp_wirelessnode:E3.5-8
- D1: device comp_wirelessnode:SOD-123F -> comp_wirelessnode:DO214-AC
- D2: device comp_wirelessnode:DO214-AC -> comp_wirelessnode:SOD-123F
- IC2: value STM8L101F2 -> DS18B20; device comp_wirelessnode:TSSOP20 -> 1wire:TO92-
- IC3: value MCP1703 -> STM8L101F2; device linear:SOT23 -> comp_wirelessnode:TSSOP20
- IC4: value DS18B20 -> MCP1703; device 1wire:TO92- -> linear:SOT23
- R10: value 47 -> 3.3k
- R16: value 10k -> 47
- R17: value 4.7k -> 47
- R18: value 47 -> 10k
- R6: value 2k -> 4.7k
- R7: value 8.6K -> 2k
- R8: value 10k -> 8.6K
- R9: value 3.3k -> 10k
- T1: value VO3063-X007T -> BTA16; device optocoupler:DIL6-SMD -> comp_wirelessnode:TO220_SMD
- moved R9 41.6 mm to (36.5, 9.26), turned to 90 degrees
- moved R17 36.6 mm to (5.80, 10.3), turned to 180 degrees
- moved IC4 31.3 mm to (14.2, 15.2), flipped to the top, turned to 0 degrees
- moved R11 29.6 mm to (38.0, 2.30), flipped to the bottom, turned to 180 degrees
- moved R10 28.4 mm to (1.96, 32.5)
- moved R6 27.6 mm to (39.9, 10.5), turned to 270 degrees
- moved R8 22.4 mm to (19.8, 24.2), turned to 270 degrees
- moved R18 21.4 mm to (21.8, 16.3), flipped to the top, turned to 270 degrees
- moved IC2 21.4 mm to (46.1, 13.9), flipped to the bottom
- moved D1 18.5 mm to (5.81, 29.2), turned to 0 degrees
- moved T1 13.7 mm to (35.5, 27.7), flipped to the top, turned to 270 degrees
- moved IC3 13.4 mm to (25.6, 8.04), turned to 90 degrees
- moved R14 10.3 mm to (12.6, 5.50), turned to 270 degrees
- moved D2 10.1 mm to (10.8, 20.4), flipped to the top, turned to 180 degrees
- moved R15 4.87 mm to (6.60, 5.50), turned to 270 degrees
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Connections:
- new net N: B1.AC2, CON1.2, CON1.3
- net +3V3: now also IC2.3, IC3.8, IC4.2, R18.2, R6.2, R9.2; no longer IC2.8, IC3.2, IC4.3, R16.2, R17.2, R8.2
- net +9.2V: now also D2.2, IC4.3, R10.2; no longer D3.2, IC3.3, R9.2
- net BTN1: now also R16.2, R18.1; no longer R14.2, R16.1
- net DQ: now also IC2.2, R11.2, R6.1; no longer IC4.2, R17.1, R18.2
- net GND: now also B1.-, D1.A, IC2.1, IC3.7, OK1.2, R10.1; no longer CON1.2, CON1.3, D2.A, IC2.7, IC3.1, R9.1, T1.2
- net L: now also R1.1, T1.1; no longer R1.2, T2.1
- net LED_TX_ERR1: now also IC3.1; no longer IC2.1
- net LED_TX_ERR2: now also IC3.2; no longer IC2.2
- net LIGHT_ON: now also IC3.10, IC3.9; no longer IC2.10, IC2.9
- net LOAD: now also T1.2; no longer T2.2
- net MISO: now also R12.2; no longer R10.2
- net MOSI: now also R13.2; no longer R11.2
- net N$10: now also B1.+; no longer D1.1
- net N$11: now also OK1.1; no longer T1.1
- net N$12: now also B1.AC1, R1.2; no longer D1.2, R1.1
- net N$13: now also IC3.15, R14.1; no longer IC2.15, R12.1
- net N$14: now also IC3.16, R13.1; no longer IC2.16, R11.1
- net N$15: now also IC3.17, R12.1; no longer IC2.17, R10.1
- net N$16: now also IC3.11, R17.1; no longer IC2.11, R15.1
- net N$17: now also IC3.13, R16.1; no longer IC2.13, R14.1
- net N$18: now also IC3.19, R11.1; no longer IC2.19, R18.1
- net N$3: now also D2.1, R8.2; no longer D3.1, R7.2
- net N$4: now also R7.2, R8.1; no longer R6.2, R7.1
- net N$6: now also D1.C, R7.1; no longer D2.C, R6.1
- net N$7: now also OK1.6; no longer T1.6
- net N$8: now also OK1.4, T1.3; no longer T1.4, T2.3
- net N$9: now also IC3.14, R15.1; no longer IC2.14, R13.1
- net NSS: now also R15.2; no longer R13.2
- net RF_RST: now also R17.2; no longer R15.2
- net RST: now also IC3.4, R9.1; no longer IC2.4, R8.1
- net SCK: now also R14.2; no longer R12.2
- net SWIM: now also IC3.3; no longer IC2.3
Routing:
- net N: track 0.00 -> 12.2 mm
- net DQ: track 16.1 -> 23.5 mm, vias 0 -> 1
- net GND: track 156.5 -> 163.3 mm, vias 9 -> 10
- net +3V3: track 58.3 -> 64.2 mm
- net L: track 20.5 -> 17.0 mm
- net N$10: track 7.03 -> 9.85 mm
- net N$12: track 1.55 -> 3.99 mm
- net N$1: track 13.4 -> 14.7 mm
- added copper zone on layer 1, net N
- added copper zone on layer 16, net N
- removed copper zone on layer 1, net GND
- removed copper zone on layer 16, net GND
Other:
- outline, holes or cut-outs redrawn
- board text added: "Wifi node R1-T1-T1 v1.0"
