File: Wireless_Node/Triac/wirelessnode_triac.sch (EAGLE design)
At the start: 45 parts, among them CON1 POWER_CONN_4, CON2 ZL321-4P, IC1 LNK304, IC2 STM8L101F2, IC3 MCP1703, T1 VO3063-X007T, T2 BTA16

Commit message: Split project into Relay and Triac based wireless node
Parts:
- added IC4: DS18B20, 1wire:DS18B20
- added R17: 4.7k, resistor:R-EU_R0603
- added R18: 47, resistor:R-EU_R0603
Connections:
- new net DQ: IC4_1W.1W, R17.1, R18.2
- new net N$18: IC2.PC1, R18.1
- net +3V3: now also IC4P.VDD, R17.2
- net GND: now also IC4P.GND
Changed lines of the file:
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@@
 <attribute name="TME_ORDER_NUMBER" value="VO3063-X007T"/>
 </part>
+<part name="GND20" library="supply" deviceset="GND" device=""/>
+<part name="+3V1" library="supply1" deviceset="+3V3" device=""/>
+<part name="IC4" library="1wire" deviceset="DS18B20" device=""/>
+<part name="R17" library="resistor" deviceset="R-EU_" device="R0603" value="4.7k"/>
+<part name="R18" library="resistor" deviceset="R-EU_" device="R0603" value="47"/>
 </parts>
 <sheets>
@@
 <attribute name="TME_ORDER_NUMBER" x="81.28" y="129.54" size="1.778" layer="96" display="off"/>
 </instance>
+<instance part="GND20" gate="1" x="124.46" y="147.32"/>
+<instance part="+3V1" gate="G$1" x="124.46" y="170.18"/>
+<instance part="IC4" gate="A" x="124.46" y="157.48"/>
+<instance part="IC4" gate="P" x="124.46" y="157.48"/>
+<instance part="IC4" gate="_1W" x="119.38" y="157.48"/>
+<instance part="R17" gate="G$1" x="109.22" y="162.56" rot="R90"/>
+<instance part="R18" gate="G$1" x="218.44" y="127"/>
 </instances>
 <busses>
@@
 <pinref part="GND3" gate="1" pin="GND"/>
 <wire x1="71.12" y1="124.46" x2="63.5" y2="124.46" width="0.1524" layer="91"/>
+</segment>
+<segment>
+<pinref part="IC4" gate="P" pin="GND"/>
+<pinref part="GND20" gate="1" pin="GND"/>
 </segment>
 </net>
@@
 <pinref part="CON2" gate="G$1" pin="1"/>
 <wire x1="208.28" y1="170.18" x2="208.28" y2="162.56" width="0.1524" layer="91"/>
+</segment>
+<segment>
+<pinref part="IC4" gate="P" pin="VDD"/>
+<pinref part="+3V1" gate="G$1" pin="+3V3"/>
+<wire x1="124.46" y1="167.64" x2="124.46" y2="165.1" width="0.1524" layer="91"/>
+<pinref part="R17" gate="G$1" pin="2"/>
+<wire x1="109.22" y1="167.64" x2="124.46" y2="167.64" width="0.1524" layer="91"/>
+<junction x="124.46" y="167.64"/>
 </segment>
 </net>
@@
 </segment>
 </net>
+<net name="DQ" class="0">
+<segment>
+<pinref part="IC4" gate="_1W" pin="1W"/>
+<wire x1="114.3" y1="157.48" x2="109.22" y2="157.48" width="0.1524" layer="91"/>
+<pinref part="R17" gate="G$1" pin="1"/>
+<wire x1="109.22" y1="157.48" x2="101.6" y2="157.48" width="0.1524" layer="91"/>
+<junction x="109.22" y="157.48"/>
+<label x="101.6" y="157.48" size="1.778" layer="95"/>
+</segment>
+<segment>
+<pinref part="R18" gate="G$1" pin="2"/>
+<wire x1="223.52" y1="127" x2="236.22" y2="127" width="0.1524" layer="91"/>
+<label x="228.6" y="127" size="1.778" layer="95"/>
+</segment>
+</net>
+<net name="N$18" class="0">
+<segment>
+<pinref part="IC2" gate="G$1" pin="PC1"/>
+<pinref part="R18" gate="G$1" pin="1"/>
+</segment>
+</net>

Commit message: Ready for production
Parts:
- removed D3: 1A/400V, comp_wirelessnode:SL1G
- removed T2: BTA16, comp_wirelessnode:BT136SMD
- added B1: B05S, rectifier:B05S
- added OK1: VO3063-X007T, optocoupler:MOC3042S
- C1: device comp_wirelessnode:C-POL-EUCAP_8X11.5_AIR -> comp_wirelessnode:C-POL-EUE3.5-8
- C4: value 4.7u/400V -> 2.2u/400V; device comp_RFSwitch_v3:C-POL-EUE5-10,5 -> comp_wirelessnode:C-POL-EUE3.5-8; TME_ORDER_NUMBER RD2G475M1012MBB -> RD2G225M0811MBB
- D1: device comp_wirelessnode:SL1G -> comp_wirelessnode:US1G-DIO; TME_ORDER_NUMBER SL1G-DIO -> US1G-DIO
- D2: device comp_wirelessnode:US1G-DIO -> comp_wirelessnode:SL1G; TME_ORDER_NUMBER US1G-DIO -> SL1G-DIO
- IC2: value STM8L101F2 -> DS18B20; device comp_wirelessnode:STM8L101F2 -> 1wire:DS18B20; TME_ORDER_NUMBER STM8L101F2P6 -> (none)
- IC3: value MCP1703 -> STM8L101F2; device linear:MCP1703CB -> comp_wirelessnode:STM8L101F2; TME_ORDER_NUMBER MCP1703T3302ECB -> STM8L101F2P6
- IC4: value DS18B20 -> MCP1703; device 1wire:DS18B20 -> linear:MCP1703CB; TME_ORDER_NUMBER (none) -> MCP1703T3302ECB
- R10: value 47 -> 3.3k; TME_ORDER_NUMBER (none) -> RC0603FR-073K3
- R16: value 10k -> 47
- R17: value 4.7k -> 47
- R18: value 47 -> 10k
- R6: value 2k -> 4.7k; TME_ORDER_NUMBER RC0603FR-072K -> (none)
- R7: value 8.6K -> 2k; TME_ORDER_NUMBER CRCW06038K66FKTABC -> RC0603FR-072K
- R8: value 10k -> 8.6K; TME_ORDER_NUMBER (none) -> CRCW06038K66FKTABC
- R9: value 3.3k -> 10k; TME_ORDER_NUMBER RC0603FR-073K3 -> (none)
- T1: value VO3063-X007T -> BTA16; device optocoupler:MOC3042S -> comp_wirelessnode:BT136SMD; TME_ORDER_NUMBER VO3063-X007T -> BTA16-600BRG
Connections:
- new net N: B1.AC2, CON1.P$2, CON1.P$3
- net +3V3: now also IC2P.VDD, IC3.VDD, IC4.VO, R18.2, R6.2, R9.2; no longer IC2.VDD, IC3.VO, IC4P.VDD, R16.2, R17.2, R8.2
- net +9.2V: now also D2.A, IC4.VI, R10.2; no longer D3.A, IC3.VI, R9.2
- net BTN1: now also R16.2, R18.1; no longer R14.2, R16.1
- net DQ: now also IC2_1W.1W, R11.2, R6.1; no longer IC4_1W.1W, R17.1, R18.2
- net GND: now also B1.-, D1.A, IC2P.GND, IC3.VSS, IC4.GND, OK1.C, R10.1; no longer CON1.P$2, CON1.P$3, D2.A, IC2.VSS, IC3.GND, IC4P.GND, R9.1, T1.C
- net L: now also R1.1, T1.A1; no longer R1.2, T2.A1
- net LED_TX_ERR1: now also IC3.PC3; no longer IC2.PC3
- net LED_TX_ERR2: now also IC3.PC4; no longer IC2.PC4
- net LIGHT_ON: now also IC3.PB0, IC3.PD0; no longer IC2.PB0, IC2.PD0
- net LOAD: now also T1.A2; no longer T2.A2
- net MISO: now also R12.2; no longer R10.2
- net MOSI: now also R13.2; no longer R11.2
- net N$10: now also B1.+; no longer D1.C
- net N$11: now also OK1.A; no longer T1.A
- net N$12: now also B1.AC1, R1.2; no longer D1.A, R1.1
- net N$13: now also IC3.PB5, R14.1; no longer IC2.PB5, R12.1
- net N$14: now also IC3.PB6, R13.1; no longer IC2.PB6, R11.1
- net N$15: now also IC3.PB7, R12.1; no longer IC2.PB7, R10.1
- net N$16: now also IC3.PB1, R17.1; no longer IC2.PB1, R15.1
- net N$17: now also IC3.PB3, R16.1; no longer IC2.PB3, R14.1
- net N$18: now also IC3.PC1, R11.1; no longer IC2.PC1, R18.1
- net N$3: now also D2.C, R8.2; no longer D3.C, R7.2
- net N$4: now also R7.2, R8.1; no longer R6.2, R7.1
- net N$6: now also D1.C, R7.1; no longer D2.C, R6.1
- net N$7: now also OK1.A2; no longer T1.A2
- net N$8: now also OK1.A1, T1.G; no longer T1.A1, T2.G
- net N$9: now also IC3.PB4, R15.1; no longer IC2.PB4, R13.1
- net NSS: now also R15.2; no longer R13.2
- net RF_RST: now also R17.2; no longer R15.2
- net RST: now also IC3.NRST/PA1, R9.1; no longer IC2.NRST/PA1, R8.1
- net SCK: now also R14.2; no longer R12.2
- net SWIM: now also IC3.PA0; no longer IC2.PA0
Other:
- moved on the sheet: D1, D2, R1, R10, R11, R12, R13, R14, R15, R16, R17, R18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
